File: hardware/electronics/mainBoard/power.kicad_sch (KiCad schematic)
At the start: 9 parts

Commit message: batt charger stuff
Parts:
- added C4: 4.7uF, symbol DSE-Passives:C
- added D2: LED, symbol Device:LED
- added R2: VAL, symbol DSE-Passives:R_horizontal
- U2: value ~ -> BQ25798RQMR
Connections:
- net GND: now also C4.2
- net at U2.1 (STAT): now also D2.1 (K)
- net at U2.5 (REGN): now also C4.1
- new net: D2.2 (A), R2.2
- new net REGN: R2.1
Other:
- moved on the sheet: C2, C3, U2

Commit message: battery management stuff
Parts:
- removed C1: 100nF, symbol DSE-Passives:C
- removed D1: ~, symbol DSE-Passives:D_Schottky
- removed Q1, Q2: ~, symbol DSE-Transistors:NMOS_GSD
- removed R1: 294R, symbol DSE-Passives:R_horizontal
- added C201, C202, C208, C209, C210, C212, C213, C214, C215, C216, C217, C218: 10uF, symbol DSE-Passives:C
- added C203, C207, C211, C225: 100nF, symbol DSE-Passives:C
- added C219: 47nF, symbol DSE-Passives:C
- added C220, C224: 100pF, symbol DSE-Passives:C
- added C221: 1uF, symbol DSE-Passives:C
- added C222, C223: 1uF, symbol DSE-Passives:C_horizontal
- added C226, C227: 100nF, symbol DSE-Passives:C_horizontal
- added C228, C229, C230: 220nF, symbol DSE-Passives:C
- added D202, D203: VAL, symbol DSE-Passives:D_Schottky_horizontal
- added D203: VAL, symbol DSE-Passives:D_Schottky
- added F201: VAL, symbol DSE-Passives:F_horizontal
- added J2: Conn_01x03_Socket, symbol Connector:Conn_01x03_Socket
- added Q201: ~, symbol DSE-Transistors:NMOS_GSD
- added Q202, Q203: VAL, symbol DSE-Transistors:NMOS_GSD
- added R202, R211: 10K, symbol DSE-Passives:R
- added R203: 8K2, symbol DSE-Passives:R_horizontal
- added R204: 127K, symbol DSE-Passives:R
- added R205: 100K, symbol DSE-Passives:R
- added R206, R209, R210, R213, R214: 100R, symbol DSE-Passives:R_horizontal
- added R207: 5K24, symbol DSE-Passives:R
- added R208: 30K31, symbol DSE-Passives:R
- added R215: 1mR, symbol DSE-Passives:R
- added R216, R219: 10M, symbol DSE-Passives:R
- added R217, R218: 5K1, symbol DSE-Passives:R
- added R220, R221, R222: 10R, symbol DSE-Passives:R_horizontal
- added TH201: 10K, symbol DSE-Passives:Thermistor
- added U3: BQ76905, symbol DSE-PMIC:BQ76905
- C204: renamed from C2; Voltage Rating VOLTAGE -> 20V
- C205: renamed from C3; Voltage Rating VOLTAGE -> 20V
- L201: renamed from L1; value 100nH -> 2.2uH
- R201: renamed from R2; value VAL -> 2K2; Package PKG -> 0603
- renumbered C4 to C206, D2 to D201
Connections:
- net GND: now also U2.10 (ACDRV2), U2.11 (ACDRV1), U2.27 (GND), C201.2, C202.2, C203.2, C207.2, C208.2, C209.2, C210.2, C211.2, C212.2, C213.2, C214.2, C215.2, C216.2, C217.2, C218.2, C219.2, C220.2, C221.2, C222.1, C223.1, C228.2, C229.2, R203.2, R205.2, R208.2, TH201.2, U3.11 (VSS), U3.21 (PGND)
- net REGN: now also R204.1, R207.1
- net VBUS: now also U2.8 (VAC2), U2.9 (VAC1), C201.1, C202.1, C203.1, F201.2
- net VIN: now also F201.1; no longer U2.9 (VAC1)
- net ~{QON}: now reaches U2.12 (~{QON})
- net ~{CE}: now reaches U2.13 (~{CE})
- net SCL: now reaches U2.14 (SCL)
- net SCL: now also U3.12 (SCL)
- net SDA: now reaches U2.15 (SDA)
- net SDA: now also U3.13 (SDA)
- net TS: now reaches U2.16 (TS)
- net TS: now also R207.2, R208.1, TH201.1, U3.8 (TS)
- net ILIM_HZ: now reaches U2.17 (ILIM_HZ)
- net ILIM_HZ: now also R204.2, R205.1
- net at U2.18 (BATP): now also C219.1, R206.1
- net at U2.20 (PROG): now also R203.1
- net BAT_CHG_INT: now reaches U2.21 (~{INT})
- net BAT_CHG_INT: now also R202.2
- net at U2.22 (BAT), U2.23 (BAT): now also C217.1, C218.1, Q201.2
- net at U2.24 (SDRV): now also Q201.1
- net at U2.25 (SYS): now also C211.1, C212.1, C213.1, C214.1, C215.1, C216.1
- net at U2.29 (PMID): now also C207.1, C208.1, C209.1, C210.1
- new net: D203.2, Q203.1, R218.2, R219.1
- new net: C227.2, D203.1, Q203.2, R219.2
- new net: Q202.1, R216.1, R217.2
- new net: C226.1, Q202.2, R214.2, R215.2, R216.2
- new net: Q202.3, Q203.3
- new net: C222.2, U3.15 (REGOUT)
- new net: C223.2, U3.16 (REGSRC)
- new net: C220.1, C221.1, R209.1, U3.17 (BAT)
- new net: C224.1, C225.1, R213.1, U3.6 (SRP)
- new net: C224.2, C225.2, R214.1, U3.7 (SRN)
- new net: C226.2, C227.1
- new net: D203.2, R210.2
- new net: D202.2, R209.2
- new net +3V3: R202.1
- new net BAL_ALERT: R211.2, U3.14 (ALERT)
- new net BAT+: D202.1, D203.1, J2.1 (Pin_1), Q201.3, R206.2, R222.1
- new net BAT-: J2.3 (Pin_3), R213.2, R215.1, R220.1
- new net BAT_1P: R221.1
- new net BAT_P1: J2.2 (Pin_2)
- new net CHG: R218.1, U3.10 (CHG)
- new net DSG: R217.1, U3.9 (DSG)
- new net REGOUT: R211.1
- new net REGSRC: R210.1
- new net VC0: C228.1, R220.2, U3.5 (VC0)
- new net VC1: C229.1, C230.2, R221.2, U3.1 (VC3A), U3.19 (VC4A), U3.2 (VC3B), U3.20 (VC4B), U3.3 (VC2), U3.4 (VC1)
- new net VC5: C230.1, R222.2, U3.18 (VC5)
Other:
- note added: "Battery Charger"
- title: Power -> Battery Charger
- moved on the sheet: C204, C205, C206, D201, L201, R201, U2
