File: hardware/electronics/mainBoard/microcontroller.kicad_sch (KiCad schematic)
At the start: 1 part, among them U1 Portenta H7

Commit message: small changes
Parts:
- removed U1: Portenta H7, symbol DSE-Micocontrollers:Portenta_H7_Mezzanine
Other:
- removed sheet Power

Commit message: working on microcontroller schematic
Parts:
- added C1: CAP, symbol DS-Passives:C_horizontal
- added R1, R3: 10K, symbol DS-Passives:R_horizontal
- added R2: 0R, symbol DS-Passives:R_horizontal
- added SW1: VAL, symbol DS-Switches:SPDT
- added SW2: VAL, symbol DS-Switches:SPST-NO Button
- added U1: STM32H745ZIT6, LQFP-144, symbol lib_sch:STM32H745ZIT6
Connections:
- new net: R3.1, U1.135 (BOOT0)
- new net: R1.1, R2.1, U1.142 (PDR_ON)
- new net: C1.1, SW2.1, SW2.4, U1.27 (NRST)
- new net: R3.2, SW1.2
- new net +3V3: R1.2, SW1.1, U1.90 (VDD50USB), U1.91 (VDD33USB)
- new net AGND: U1.34 (VSSA)
- new net VCAP: U1.103 (VCAP), U1.140 (VCAP), U1.68 (VCAP)
- new net VDD: U1.106 (VDD), U1.119 (VDD), U1.129 (VDD), U1.13 (VDD), U1.144 (VDD), U1.19 (VDD), U1.32 (VDD), U1.35 (VREF+), U1.36 (VDDA), U1.42 (VDD), U1.56 (VDD), U1.7 (VDD), U1.71 (VDD), U1.79 (VDD), U1.8 (VBAT), U1.92 (VDD)
- new net VDD_LDO: U1.105 (VDDLDO), U1.143 (VDDLDO), U1.70 (VDDLDO)
- new net VDD_SMPS_IN: U1.16 (VDDSMPS)
- new net VDD_SMPS_OUT: U1.15 (VLXSMPS)
- new net VFBSD: U1.17 (VFBSMPS)
- new net VSS: C1.2, R2.2, SW1.3, SW2.2, SW2.3, U1.104 (VSS), U1.118 (VSS), U1.12 (VSS), U1.128 (VSS), U1.14 (VSSSMPS), U1.141 (VSS), U1.18 (VSS), U1.33 (VSS), U1.41 (VSS), U1.55 (VSS), U1.6 (VSS), U1.69 (VSS), U1.80 (VSS), U1.89 (VSS)
Other:
- title: (none) -> Microcontroller
