File: hardware/electronics/mainBoard/stm32h745_power_supplies.kicad_sch (KiCad schematic)
At the start: 34 parts, among them U1 STM32H745ZIT6

Commit message: power supplies for H745
Parts:
- C10, C11, C12, C13, C14, C15, C16, C17, C18, C19, C20, C21, C22, C23, C24, C25, C26, C27, C4, C5, C6, C7, C8, C9: symbol DS-Passives:C -> lib_sch:C
- L1: symbol DS-Passives:Ferrite_horizontal -> lib_sch:Ferrite_horizontal
- L2: symbol DS-Passives:L_horizontal -> lib_sch:L_horizontal
- NT2, NT3, NT4, NT5, NT6, NT7: symbol Device:NetTie_2 -> lib_sch:NetTie_2
- R4: symbol DS-Passives:R_horizontal -> lib_sch:R_horizontal

Commit message: fixed inductor
Parts:
- L2: footprint (none) -> lib_fp:WE-XHMI-4030; Current Rating IMAX -> 7A8; DC Resistance DCR -> 19.8mR; DKPN (none) -> 732-74439324022CT-ND; MPN (none) -> 74439324022; Manufacturer (none) -> Würth Elektronik; Resonant Frequency FRES -> 40MHz; Tolerance TOL -> 20%
Changed lines of the file:
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@@
 	(title_block
 		(title "STM32H745 Power Supplies")
-		(date "2025-02-24")
+		(date "2025-03-03")
 		(rev "1")
 		(comment 2 "PROTOTYPE")
@@
 			)
 		)
-		(property "Footprint" ""
+		(property "Footprint" "lib_fp:WE-XHMI-4030"
 			(at 119.38 173.99 0)
 			(effects
@@
 			)
 		)
-		(property "Datasheet" ""
+		(property "Datasheet" "datasheets/Wurth-Elektronik-74439324022.pdf"
 			(at 119.38 173.99 0)
 			(effects
@@
 			)
 		)
-		(property "Description" ""
+		(property "Description" "2.2 µH Shielded Molded Inductor 7.8 A 19.8mOhm Max Nonstandard"
 			(at 120.65 173.99 0)
 			(effects
@@
 			)
 		)
-		(property "Manufacturer" ""
+		(property "Manufacturer" "Würth Elektronik"
 			(at 120.65 173.99 0)
 			(effects
@@
 			)
 		)
-		(property "MPN" ""
+		(property "MPN" "74439324022"
 			(at 120.65 173.99 0)
 			(effects
@@
 			)
 		)
-		(property "DKPN" ""
+		(property "DKPN" "732-74439324022CT-ND"
 			(at 120.65 173.99 0)
 			(effects
@@
 			)
 		)
-		(property "Tolerance" "TOL"
+		(property "Tolerance" "20%"
 			(at 120.65 174.879 0)
 			(do_not_autoplace yes)
@@
 			)
 		)
-		(property "Current Rating" "IMAX"
+		(property "Current Rating" "7A8"
 			(at 120.65 174.879 0)
 			(do_not_autoplace yes)
@@
 			)
 		)
-		(property "DC Resistance" "DCR"
+		(property "DC Resistance" "19.8mR"
 			(at 120.65 175.895 0)
 			(do_not_autoplace yes)
@@
 			)
 		)
-		(property "Resonant Frequency" "FRES"
+		(property "Resonant Frequency" "40MHz"
 			(at 120.65 175.895 0)
 			(do_not_autoplace yes)
