File: hardware/electronics/mainBoard/mainBoard.kicad_pcb (KiCad board)
At the start: 4 copper layers, 160 x 100 mm, 0 parts

Commit message: assigned footprints
Parts:
- added AE1: TNC, lib_connectors:RFPC-TNC01-FN, F.Cu at (238.0, 117.2)
- added AE2: SMA, lib_connectors:RFPC-SMA14-FN, F.Cu at (253.0, 106.1)
- added AE3: SMA, lib_connectors:RFPC-SMA14-FN, F.Cu at (265.1, 106.1)
- added C1: 4.7uF, lib_passives:GCM0805, F.Cu at (-58.3, 109.9)
- added C10: 100nF, lib_passives:GCM0402, F.Cu at (-88.5, 136.5)
- added C100: 100nF, lib_passives:GCM0402, F.Cu at (-84.5, 49.8)
- added C101: 10uF, lib_passives:GRT1210, F.Cu at (-64.8, 23.3)
- added C102: 10uF, lib_passives:GRT1210, F.Cu at (-64.8, 27.8)
- added C103: 10uF, lib_passives:GRT1210, F.Cu at (-58.5, 14.4)
- added C104: 10uF, lib_passives:GRT1210, F.Cu at (-58.5, 18.9)
- added C105: 10uF, lib_passives:GRT1210, F.Cu at (-58.5, 23.3)
- added C106: 10uF, lib_passives:GRT1210, F.Cu at (-58.5, 27.8)
- added C107: 10uF, lib_passives:GRT1210, F.Cu at (-52.3, 14.4)
- added C108: 10uF, lib_passives:GRT1210, F.Cu at (-52.3, 18.9)
- added C109: 10uF, lib_passives:GRT1210, F.Cu at (-52.3, 23.3)
- added C11: 100nF, lib_passives:GCM0402, F.Cu at (-88.5, 138.6)
- added C110: 10uF, lib_passives:GRT1210, F.Cu at (-52.3, 27.8)
- added C111: 220nF, lib_passives:GCM0402, F.Cu at (-19.1, 111.5)
- added C112: 220nF, lib_passives:GCM0402, F.Cu at (-19.1, 113.6)
- added C113: 220nF, lib_passives:GCM0402, F.Cu at (-19.1, 115.7)
- added C114: 2.2uF, lib_passives:GCM0805, F.Cu at (-18.0, 102.8)
- added C115: 100nF, lib_passives:GCM0402, F.Cu at (-19.1, 117.8)
- added C116: 100pF, lib_passives:GCM0402, F.Cu at (-19.1, 119.9)
- added C117: 100pF, lib_passives:GCM0402, F.Cu at (-16.0, 111.5)
- added C118: 1uF, lib_passives:GRT0603, F.Cu at (-37.8, 119.2)
- added C119: 2.2uF, lib_passives:GCM0805, F.Cu at (-18.0, 105.7)
- added C12: 100nF, lib_passives:GCM0402, F.Cu at (-88.5, 140.7)
- added C120: 100nF, lib_passives:GCM0402, F.Cu at (-16.0, 113.6)
- added C121: 100nF, lib_passives:GCM0402, F.Cu at (-16.0, 115.7)
- added C122: 100nF, lib_passives:GCM0402, F.Cu at (-16.0, 117.8)
- added C123: 100nF, lib_passives:GCM0402, F.Cu at (-16.0, 119.9)
- added C124: 4.7uF, lib_passives:GCM0805, F.Cu at (-13.2, 41.5)
- added C125: 2.2uF, lib_passives:GCM0805, F.Cu at (-13.2, 44.4)
- added C126: 150pF, lib_passives:GCM0402, F.Cu at (-9.47, 41.1)
- added C127: 10uF, lib_passives:GCM0805, F.Cu at (-13.2, 47.3)
- added C128: 3.9nF, lib_passives:GCM0402, F.Cu at (-9.47, 43.2)
- added C129: 100nF, lib_passives:GCM0402, F.Cu at (-9.47, 45.3)
- added C13: 100nF, lib_passives:GCM0402, F.Cu at (-88.5, 142.8)
- added C130: 100nF, lib_passives:GCM0402, F.Cu at (-9.47, 47.5)
- added C131: 22uF, lib_passives:GCM1206, F.Cu at (-11.6, 13.8)
- added C132: 22uF, lib_passives:GCM1206, F.Cu at (-11.6, 17.1)
- added C133: 22uF, lib_passives:GCM1206, F.Cu at (-11.6, 20.4)
- added C134: 22uF, lib_passives:GCM1206, F.Cu at (-11.6, 23.6)
- added C14: 100nF, lib_passives:GCM0402, F.Cu at (-88.5, 144.9)
- added C15: 220pF, lib_passives:GCM0402, F.Cu at (-88.5, 147.1)
- added C16: 1uF, lib_passives:GRT0603, F.Cu at (-58.6, 124.4)
- added C17: 4.7uF, lib_passives:GCM0805, F.Cu at (-58.3, 112.8)
- added C18: 100nF, lib_passives:GCM0402, F.Cu at (-85.5, 134.4)
- added C19: 10uF, lib_passives:GCM0805, F.Cu at (-58.3, 115.7)
- added C2: 100nF, lib_passives:GCM0402, F.Cu at (-91.5, 134.4)
- added C20: 1uF, lib_passives:GRT0603, F.Cu at (-58.6, 126.9)
- added C21: 100nF, lib_passives:GCM0402, F.Cu at (-85.5, 136.5)
- added C22: 100nF, lib_passives:GCM0402, F.Cu at (-85.5, 138.6)
- added C23: 100nF, lib_passives:GCM0402, F.Cu at (-85.5, 140.7)
- added C24: 100nF, lib_passives:GCM0402, F.Cu at (-85.5, 142.8)
- added C25: 100nF, lib_passives:GCM0402, F.Cu at (-85.5, 144.9)
- added C26: 100nF, lib_passives:GCM0402, F.Cu at (-85.5, 147.1)
- added C27: 100nF, lib_passives:GCM0402, F.Cu at (-21.2, 139.3)
- added C28: 100nF, lib_passives:GCM0402, F.Cu at (-21.2, 141.4)
- added C29: 100nF, lib_passives:GCM0402, F.Cu at (-21.2, 143.6)
- added C3: 100nF, lib_passives:GCM0402, F.Cu at (-91.5, 136.5)
- added C30: 100nF, lib_passives:GCM0402, F.Cu at (30.2, 110.9)
- added C31: 100nF, lib_passives:GCM0402, F.Cu at (30.2, 113.0)
- added C32: 100nF, lib_passives:GCM0402, F.Cu at (30.2, 115.1)
- added C33: 10uF, lib_passives:GCM0805, F.Cu at (5.29, 82.3)
- added C34: 100nF, lib_passives:GCM0402, F.Cu at (26.7, 67.2)
- added C35: 100nF, lib_passives:GCM0402, F.Cu at (26.7, 69.3)
- added C36: 470pF, lib_passives:GCM0402, F.Cu at (26.7, 71.4)
- added C37: 1uF, lib_passives:GRT0603, F.Cu at (9.49, 82.1)
- added C38: 100nF, lib_passives:GCM0402, F.Cu at (26.7, 73.5)
- added C39: 100nF, lib_passives:GCM0402, F.Cu at (26.7, 75.7)
- added C4: 100nF, lib_passives:GCM0402, F.Cu at (-91.5, 138.6)
- added C40: 1uF, lib_passives:GRT0603, F.Cu at (33.9, 90.6)
- added C41: 1uF, lib_passives:GRT0603, F.Cu at (33.9, 93.1)
- added C42: 1uF, lib_passives:GRT0603, F.Cu at (33.9, 95.6)
- added C43: 1uF, lib_passives:GRT0603, F.Cu at (33.9, 98.1)
- added C44: 100nF, lib_passives:GCM0402, F.Cu at (26.4, 100.5)
- added C45: 100nF, lib_passives:GCM0402, F.Cu at (26.4, 102.6)
- added C46: 100nF, lib_passives:GCM0402, F.Cu at (26.4, 104.7)
- added C47: 100nF, lib_passives:GCM0402, F.Cu at (26.4, 106.8)
- added C48: 100nF, lib_passives:GCM0402, F.Cu at (6.95, 101.6)
- added C49: 100nF, lib_passives:GCM0402, F.Cu at (6.95, 103.8)
- added C5: 100nF, lib_passives:GCM0402, F.Cu at (-91.5, 140.7)
- added C50: 100nF, lib_passives:GCM0402, F.Cu at (6.95, 105.9)
- added C51: 100nF, lib_passives:GCM0402, F.Cu at (6.95, 108.0)
- added C52: 1uF, lib_passives:GRT0603, F.Cu at (10.4, 118.9)
- added C53: 1uF, lib_passives:GRT0603, F.Cu at (10.4, 121.4)
- added C54: 100nF, lib_passives:GCM0402, F.Cu at (6.95, 110.1)
- added C55: 100nF, lib_passives:GCM0402, F.Cu at (6.95, 112.2)
- added C56: 100nF, lib_passives:GCM0402, F.Cu at (6.95, 114.3)
- added C57: 100nF, lib_passives:GCM0402, F.Cu at (-27.5, 63.7)
- added C58: 100nF, lib_passives:GCM0402, F.Cu at (-27.5, 65.8)
- added C59: 100nF, lib_passives:GCM0402, F.Cu at (-27.5, 67.9)
- added C6: 100nF, lib_passives:GCM0402, F.Cu at (-91.5, 142.8)
- added C60: 100nF, lib_passives:GCM0402, F.Cu at (-27.5, 70.0)
- added C61: 1uF, lib_passives:GRT0603, F.Cu at (-14.0, 83.6)
- added C62: 1uF, lib_passives:GRT0603, F.Cu at (-14.0, 86.1)
- added C63: 100nF, lib_passives:GCM0402, F.Cu at (-27.5, 72.2)
- added C64: 100nF, lib_passives:GCM0402, F.Cu at (-27.5, 74.3)
- added C65: 100nF, lib_passives:GCM0402, F.Cu at (-27.5, 76.4)
- added C66: 100nF, lib_passives:GCM0402, F.Cu at (14.9, 24.5)
- added C67: 100nF, lib_passives:GCM0402, F.Cu at (14.9, 26.6)
- added C68: 100nF, lib_passives:GCM0402, F.Cu at (14.9, 28.8)
- added C69: 100nF, lib_passives:GCM0402, F.Cu at (14.9, 30.9)
- added C7: 100nF, lib_passives:GCM0402, F.Cu at (-91.5, 144.9)
- added C70: 1uF, lib_passives:GRT0603, F.Cu at (28.4, 44.4)
- added C71: 1uF, lib_passives:GRT0603, F.Cu at (28.4, 46.9)
- added C72: 100nF, lib_passives:GCM0402, F.Cu at (14.9, 33.0)
- added C73: 100nF, lib_passives:GCM0402, F.Cu at (14.9, 35.1)
- added C74: 100nF, lib_passives:GCM0402, F.Cu at (14.9, 37.2)
- added C75: 9.1pF, lib_passives:GCM0402, F.Cu at (-68.1, 85.3)
- added C76: 100pF, lib_passives:GCM0402, F.Cu at (-68.1, 87.4)
- added C77: 5.6pF, lib_passives:GCM0402, F.Cu at (-68.1, 89.5)
- added C78: 100pF, lib_passives:GCM0402, F.Cu at (-68.1, 91.6)
- added C79: 100nF, lib_passives:GCM0402, F.Cu at (-68.1, 93.7)
- added C8: 100nF, lib_passives:GCM0402, F.Cu at (-91.5, 147.1)
- added C80: 100nF, lib_passives:GCM0402, F.Cu at (-68.1, 95.8)
- added C81: 9.1pF, lib_passives:GCM0402, F.Cu at (-68.1, 97.9)
- added C82: 100nF, lib_passives:GCM0402, F.Cu at (-1.30, 152.1)
- added C83: 10uF, lib_passives:GCM0805, F.Cu at (26.6, 148.5)
- added C84: 4.7uF, lib_passives:GCM0805, F.Cu at (26.6, 151.4)
- added C85: 1uF, lib_passives:GRT0603, F.Cu at (37.1, 139.0)
- added C86: 100nF, lib_passives:GCM0402, F.Cu at (35.6, 141.3)
- added C87: 100nF, lib_passives:GCM0402, F.Cu at (35.6, 143.4)
- added C88: 100nF, lib_passives:GCM0402, F.Cu at (35.6, 145.6)
- added C89: 100nF, lib_passives:GCM0402, F.Cu at (35.6, 147.7)
- added C9: 100nF, lib_passives:GCM0402, F.Cu at (-88.5, 134.4)
- added C90: 100nF, lib_passives:GCM0402, F.Cu at (-84.5, 35.1)
- added C91: 100nF, lib_passives:GCM0402, F.Cu at (-84.5, 37.2)
- added C92: 47nF, lib_passives:GCM0402, F.Cu at (-84.5, 39.3)
- added C93: 47nF, lib_passives:GCM0402, F.Cu at (-84.5, 41.4)
- added C94: 10uF, lib_passives:GRT1210, F.Cu at (-64.8, 14.4)
- added C95: 10uF, lib_passives:GRT1210, F.Cu at (-64.8, 18.9)
- added C96: 100nF, lib_passives:GCM0402, F.Cu at (-84.5, 43.5)
- added C97: 4.7uF, lib_passives:GCM0805, F.Cu at (-71.6, 58.7)
- added C98: 47nF, lib_passives:GCM0402, F.Cu at (-84.5, 45.6)
- added C99: 100nF, lib_passives:GCM0402, F.Cu at (-84.5, 47.7)
- added D1: LTST-C191KRKT, lib_diodes:LTST-0603, F.Cu at (-58.5, 129.4)
- added D10: LTST-C191TBKT, lib_diodes:LTST-0603, F.Cu at (24.9, 13.5)
- added D11: LTST-C191KRKT, lib_diodes:LTST-0603, F.Cu at (24.9, 16.0)
- added D12: LTST-C191KGKT, lib_diodes:LTST-0603, F.Cu at (24.9, 18.6)
- added D13: LTST-C191KRKT, lib_diodes:LTST-0603, F.Cu at (33.1, 139.0)
- added D14: D1213A-01LP4, lib_diodes:XDFN2P65_100X60X50L50X25L, F.Cu at (35.5, 149.8)
- added D15: BZT52C12T-7, lib_diodes:SOD523, F.Cu at (-50.7, 55.4)
- added D16: BZT52C12T-7, lib_diodes:SOD523, F.Cu at (-50.7, 57.8)
- added D17: LTST-C191KGKT, lib_diodes:LTST-0603, F.Cu at (-65.9, 31.3)
- added D18: SDM20U40Q-7, lib_diodes:SOD523, F.Cu at (-41.4, 119.2)
- added D19: SDM20U40Q-7, lib_diodes:SOD523, F.Cu at (-41.4, 121.5)
- added D2: D1213A-01LP4, lib_diodes:XDFN2P65_100X60X50L50X25L, F.Cu at (-60.4, 143.7)
- added D20: MMSZ5246B-7-F, lib_diodes:SOD123, F.Cu at (-17.4, 108.7)
- added D21: LTST-C191KRKT, lib_diodes:LTST-0603, F.Cu at (-44.1, 44.4)
- added D22: LTST-C191KRKT, lib_diodes:LTST-0603, F.Cu at (-44.1, 47.0)
- added D3: USBLC6-4SC6, lib_ICs:SOT2395P280X145-6, F.Cu at (0.57, 83.0)
- added D4: LTST-C191TBKT, lib_diodes:LTST-0603, F.Cu at (17.0, 90.6)
- added D5: LTST-C191KRKT, lib_diodes:LTST-0603, F.Cu at (17.0, 93.1)
- added D6: LTST-C191KGKT, lib_diodes:LTST-0603, F.Cu at (17.0, 95.7)
- added D7: LTST-C191TBKT, lib_diodes:LTST-0603, F.Cu at (-17.5, 52.7)
- added D8: LTST-C191KRKT, lib_diodes:LTST-0603, F.Cu at (-17.5, 55.2)
- added D9: LTST-C191KGKT, lib_diodes:LTST-0603, F.Cu at (-17.5, 57.8)
- added J1: Chassis Ground Strap, lib_connectors:M4.5-MH, F.Cu at (38.8, 114.9)
- added J10: M.2 Standoff, lib_connectors:M4.5-MH, F.Cu at (-34.1, 77.7)
- added J11: M.2 Standoff, lib_connectors:M4.5-MH, F.Cu at (8.39, 28.5)
- added J12: Bus_M.2_Socket_E, lib_connectors:MDT420E01001, F.Cu at (8.09, 19.7)
- added J13: M.2 Standoff, lib_connectors:M4.5-MH, F.Cu at (8.39, 38.6)
- added J14: CONMHF1-SMD-T, lib_connectors:CONMHF1, F.Cu at (-72.4, 87.0)
- added J15: CONMHF1-SMD-T, lib_connectors:CONMHF1, F.Cu at (-72.4, 92.5)
- added J16: CONMHF1-SMD-T, lib_connectors:CONMHF1, F.Cu at (-72.4, 98.1)
- added J17: CONMHF1-SMD-T, lib_connectors:CONMHF1, F.Cu at (-72.4, 103.6)
- added J18: STEMMA-QT, lib_connectors:JST_SH_BM04B-SRSS-TB, F.Cu at (-7.24, 127.8)
- added J19: M8S-04PFFR-SF8001, lib_connectors:M8S-04PFFR-SF8001, F.Cu at (79.5, 76.9)
- added J2: ~, lib_misc:TC2050-FP, F.Cu at (-77.5, 139.9)
- added J20: STEMMA-QT, lib_connectors:JST_SH_BM04B-SRSS-TB, F.Cu at (-7.24, 134.1)
- added J21: STEMMA-QT, lib_connectors:JST_SH_BM04B-SRSS-TB, F.Cu at (-7.24, 140.3)
- added J22: STEMMA-QT, lib_connectors:JST_SH_BM04B-SRSS-TB, F.Cu at (-7.24, 146.6)
- added J23: STEMMA-QT, lib_connectors:JST_SH_BM04B-SRSS-TB, F.Cu at (-7.24, 152.8)
- added J24: ~, lib_misc:TC2050-FP, F.Cu at (23.8, 131.2)
- added J25: M8AS-02PFFR-SF8001, lib_connectors:M8AS-02PFFR-SF8001, F.Cu at (79.5, 59.2)
- added J26: MUSBRM1C1M0, lib_connectors:MUSBR-M1C1-XX, F.Cu at (72.4, 100.3)
- added J27: S2B-PH-SM4-TB, lib_connectors:JST-PH-S2B-SM4-TB, F.Cu at (-53.3, 40.6)
- added J28: 1726480102, lib_connectors:1726480102, F.Cu at (-40.8, 94.8)
- added J29: S3B-XH-SM4-TB, lib_connectors:JST_XH_S3B-SM4-TB, F.Cu at (-28.3, 95.3)
- added J3: MEM2067-02-180-00-A, lib_connectors:MEM2067-02-180-00-A, F.Cu at (-37.9, 125.9)
- added J30: Conn_01x04_Pin, lib_connectors:conn_01x04_254_right_angle, F.Cu at (-39.6, 14.0)
- added J31: Conn_01x04_Pin, lib_connectors:conn_01x04_254_right_angle, F.Cu at (-39.6, 26.3)
- added J4: MRJ-5381-01, lib_connectors:MJR-5381-X1, F.Cu at (76.5, 132.9)
- added J5: M.2 Standoff, lib_connectors:M4.5-MH, F.Cu at (0.41, 105.6)
- added J6: Bus_M.2_Socket_E, lib_connectors:MDT420E01001, F.Cu at (0.11, 96.8)
- added J7: M.2 Standoff, lib_connectors:M4.5-MH, F.Cu at (0.80, 117.3)
- added J8: M.2 Standoff, lib_connectors:M4.5-MH, F.Cu at (-34.1, 67.7)
- added J9: Bus_M.2_Socket_E, lib_connectors:MDT420E01001, F.Cu at (-34.4, 58.8)
- added JP1: ~, lib_misc:SolderJumper-2_P1.3mm_Bridged_RoundedPad1.0x1.5mm, F.Cu at (20.7, 108.4)
- added JP10: ~, lib_misc:SolderJumper-2_P1.3mm_Bridged_RoundedPad1.0x1.5mm, F.Cu at (-64.1, 57.9)
- added JP11: ~, lib_misc:SolderJumper-3_P1.3mm_Bridged12_RoundedPad1.0x1.5mm, F.Cu at (-25.9, 47.3)
- added JP12: ~, lib_misc:SolderJumper-2_P1.3mm_Bridged_RoundedPad1.0x1.5mm, F.Cu at (-30.9, 43.1)
- added JP13: ~, lib_misc:SolderJumper-2_P1.3mm_Bridged_RoundedPad1.0x1.5mm, F.Cu at (-30.9, 46.6)
- added JP2: ~, lib_misc:SolderJumper-2_P1.3mm_Bridged_RoundedPad1.0x1.5mm, F.Cu at (20.7, 111.9)
- added JP3: ~, lib_misc:SolderJumper-2_P1.3mm_Bridged_RoundedPad1.0x1.5mm, F.Cu at (20.7, 115.5)
- added JP4: ~, lib_misc:SolderJumper-2_P1.3mm_Bridged_RoundedPad1.0x1.5mm, F.Cu at (-13.8, 73.4)
- added JP5: ~, lib_misc:SolderJumper-2_P1.3mm_Bridged_RoundedPad1.0x1.5mm, F.Cu at (-13.8, 77.0)
- added JP6: ~, lib_misc:SolderJumper-2_P1.3mm_Bridged_RoundedPad1.0x1.5mm, F.Cu at (-13.8, 80.5)
- added JP7: ~, lib_misc:SolderJumper-2_P1.3mm_Bridged_RoundedPad1.0x1.5mm, F.Cu at (28.7, 34.3)
- added JP8: ~, lib_misc:SolderJumper-2_P1.3mm_Bridged_RoundedPad1.0x1.5mm, F.Cu at (28.7, 37.8)
- added JP9: ~, lib_misc:SolderJumper-2_P1.3mm_Bridged_RoundedPad1.0x1.5mm, F.Cu at (28.7, 41.4)
- added L1: Ferrite, lib_passives:L_0603, F.Cu at (-58.6, 131.9)
- added L2: 2.2uH, lib_passives:WE-XHMI-4030, F.Cu at (-57.5, 120.1)
- added L3: Ferrite, lib_passives:L_0603, F.Cu at (9.47, 84.6)
- added L4: 6.8nH, lib_passives:L_0603, F.Cu at (-56.7, 85.4)
- added L5: 15nH, lib_passives:L_0603, F.Cu at (-56.7, 87.9)
- added L6: 2.2uH, lib_passives:WE-XHMI-4030, F.Cu at (-63.2, 53.1)
- added L7: 1uH, lib_passives:WE-XHMI-8080, F.Cu at (-27.8, 36.0)
- added L8: 6.8uH, lib_passives:WE-XHMI-1510, F.Cu at (128.4, 73.0)
- added NT1: NetTie, lib_misc:NetTie-2_SMD_Pad2.0mm, F.Cu at (-64.3, 110.2)
- added NT10: NetTie, lib_misc:NetTie-2_SMD_Pad2.0mm, F.Cu at (-17.4, 94.6)
- added NT2: NetTie, lib_misc:NetTie-2_SMD_Pad2.0mm, F.Cu at (-64.3, 113.7)
- added NT3: NetTie, lib_misc:NetTie-2_SMD_Pad2.0mm, F.Cu at (-64.3, 117.3)
- added NT4: NetTie, lib_misc:NetTie-2_SMD_Pad2.0mm, F.Cu at (-64.3, 120.8)
- added NT5: NetTie, lib_misc:NetTie-2_SMD_Pad2.0mm, F.Cu at (-64.3, 124.4)
- added NT6: NetTie, lib_misc:NetTie-2_SMD_Pad2.0mm, F.Cu at (-64.3, 127.9)
- added NT7: NetTie, lib_misc:NetTie-2_SMD_Pad2.0mm, F.Cu at (-70.0, 51.9)
- added NT8: NetTie, lib_misc:NetTie-2_SMD_Pad2.0mm, F.Cu at (-70.0, 55.4)
- added NT9: NetTie, lib_misc:NetTie-2_SMD_Pad2.0mm, F.Cu at (-17.4, 91.1)
- added Q1: CSD17581Q3A, lib_ICs:SON65P300X315X90-8, F.Cu at (-90.2, 39.8)
- added Q10: BSS138-7-F, lib_ICs:SOT23, F.Cu at (-8.17, 32.8)
- added Q11: BSS138-7-F, lib_ICs:SOT23, F.Cu at (-8.17, 37.3)
- added Q2: CSD17581Q3A, lib_ICs:SON65P300X315X90-8, F.Cu at (-90.2, 44.4)
- added Q3: CSD17581Q3A, lib_ICs:SON65P300X315X90-8, F.Cu at (-90.2, 49.1)
- added Q4: CSD17581Q3A, lib_ICs:SON65P300X315X90-8, F.Cu at (-90.2, 53.7)
- added Q5: CSD17581Q3A, lib_ICs:SON65P300X315X90-8, F.Cu at (-90.2, 58.4)
- added Q6: BUK6D72-30EX, lib_ICs:UDFN6P65_200X200X65L30X25N, F.Cu at (-40.9, 112.7)
- added Q7: BUK6D72-30EX, lib_ICs:UDFN6P65_200X200X65L30X25N, F.Cu at (-40.9, 116.2)
- added Q8: CSD17581Q3A, lib_ICs:SON65P300X315X90-8, F.Cu at (-12.6, 33.1)
- added Q9: CSD17581Q3A, lib_ICs:SON65P300X315X90-8, F.Cu at (-12.6, 37.7)
- added R1: 47R, lib_passives:CRCW0402, F.Cu at (-69.4, 134.4)
- added R10: 4K7, lib_passives:CRCW0402, F.Cu at (-66.3, 142.8)
- added R11: 10K, lib_passives:CRCW0402, F.Cu at (-63.3, 134.4)
- added R12: 0R, lib_passives:CRCW0402, F.Cu at (-63.3, 136.5)
- added R13: 10K, lib_passives:CRCW0402, F.Cu at (-63.3, 138.6)
- added R14: 10K, lib_passives:CRCW0402, F.Cu at (-63.3, 140.7)
- added R15: 33R, lib_passives:CRCW0402, F.Cu at (23.7, 52.5)
- added R16: 33R, lib_passives:CRCW0402, F.Cu at (23.7, 54.6)
- added R17: 10K, lib_passives:CRCW0402, F.Cu at (23.7, 56.7)
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Other:
- outline, holes or cut-outs redrawn

Commit message: added board-edge keepout for enclosure rails and repositioned IO/RF connectors
Parts:
- added R92: 200K, lib_passives:CRCW0402, F.Cu at (1.03, 0.56)
- added R93: 499K, lib_passives:CRCW0402, F.Cu at (1.03, 2.67)
- added R94: 100K, lib_passives:CRCW0402, F.Cu at (1.03, 4.78)
- C1, C124, C17: value 4.7uF -> 100nF; footprint lib_passives:GCM0805 -> lib_passives:GCM0402
- C10, C12, C38, C44, C45, C48, C57, C66: value 100nF -> 1uF; footprint lib_passives:GCM0402 -> lib_passives:GRT0603
- C100, C91, C96: value 100nF -> 10uF; footprint lib_passives:GCM0402 -> lib_passives:GRT1210
- C105, C108, C109: value 10uF -> 47nF; footprint lib_passives:GRT1210 -> lib_passives:GCM0402
- C110: value 10uF -> 4.7uF; footprint lib_passives:GRT1210 -> lib_passives:GCM0805
- C115, C80: value 100nF -> 100pF
- C116: value 100pF -> 2.2uF; footprint lib_passives:GCM0402 -> lib_passives:GCM0805
- C117: value 100pF -> 1uF; footprint lib_passives:GCM0402 -> lib_passives:GRT0603
- C118, C16, C20, C42, C43, C53, C62, C71: value 1uF -> 100nF; footprint lib_passives:GRT0603 -> lib_passives:GCM0402
- C119: value 2.2uF -> 100pF; footprint lib_passives:GCM0805 -> lib_passives:GCM0402
- C125: value 2.2uF -> 4.7uF
- C126: value 150pF -> 22uF; footprint lib_passives:GCM0402 -> lib_passives:GCM1206
- C127: value 10uF -> 22uF; footprint lib_passives:GCM0805 -> lib_passives:GCM1206
- C128: value 3.9nF -> 22uF; footprint lib_passives:GCM0402 -> lib_passives:GCM1206
- C129: value 100nF -> 2.2uF; footprint lib_passives:GCM0402 -> lib_passives:GCM0805
- C131: value 22uF -> 150pF; footprint lib_passives:GCM1206 -> lib_passives:GCM0402
- C132: value 22uF -> 3.9nF; footprint lib_passives:GCM1206 -> lib_passives:GCM0402
- C133: value 22uF -> 10uF; footprint lib_passives:GCM1206 -> lib_passives:GCM0805
- C15: value 220pF -> 100nF
- C19: value 10uF -> 100nF; footprint lib_passives:GCM0805 -> lib_passives:GCM0402
- C21, C3: value 100nF -> 4.7uF; footprint lib_passives:GCM0402 -> lib_passives:GCM0805
- C23: value 100nF -> 220pF
- C24: value 100nF -> 10uF; footprint lib_passives:GCM0402 -> lib_passives:GCM0805
- C36: value 470pF -> 100nF
- C37: value 1uF -> 470pF; footprint lib_passives:GRT0603 -> lib_passives:GCM0402
- C75: value 9.1pF -> 100nF
- C76: value 100pF -> 100nF
- C77: value 5.6pF -> 9.1pF
- C78: value 100pF -> 5.6pF
- C79: value 100nF -> 9.1pF
- C81: value 9.1pF -> 100pF
- C92: value 47nF -> 10uF; footprint lib_passives:GCM0402 -> lib_passives:GRT1210
- C93, C98: value 47nF -> 100nF
- C94: value 10uF -> 100nF; footprint lib_passives:GRT1210 -> lib_passives:GCM0402
- C97: value 4.7uF -> 10uF; footprint lib_passives:GCM0805 -> lib_passives:GRT1210
- D10, D4, D7: value LTST-C191TBKT -> LTST-C191KGKT
- D11, D5, D8: value LTST-C191KRKT -> LTST-C191TBKT
- D12, D6, D9: value LTST-C191KGKT -> LTST-C191KRKT
- J1: footprint lib_connectors:M4.5-MH -> lib_misc:M4.5-MH
- J10, J13, J7: footprint lib_connectors:M4.5-MH -> lib_misc:MountingHole_3.5mm_Pad_Via
- J11, J5, J8: value M.2 Standoff -> Bus_M.2_Socket_E; footprint lib_connectors:M4.5-MH -> lib_connectors:MDT420E01001
- J12, J6, J9: value Bus_M.2_Socket_E -> M.2 Standoff; footprint lib_connectors:MDT420E01001 -> lib_misc:MountingHole_3.5mm_Pad_Via
- J18: value STEMMA-QT -> M8S-04PFFR-SF8001; footprint lib_connectors:JST_SH_BM04B-SRSS-TB -> lib_connectors:M8S-04PFFR-SF8001
- J19: value M8S-04PFFR-SF8001 -> STEMMA-QT; footprint lib_connectors:M8S-04PFFR-SF8001 -> lib_connectors:JST_SH_BM04B-SRSS-TB
- J28: value 1726480102 -> S3B-XH-SM4-TB; footprint lib_connectors:1726480102 -> lib_connectors:JST_XH_S3B-SM4-TB
- J29: value S3B-XH-SM4-TB -> 1726480102; footprint lib_connectors:JST_XH_S3B-SM4-TB -> lib_connectors:1726480102
- JP11: footprint lib_misc:SolderJumper-3_P1.3mm_Bridged12_RoundedPad1.0x1.5mm -> lib_misc:SolderJumper-2_P1.3mm_Bridged_RoundedPad1.0x1.5mm
- JP12: footprint lib_misc:SolderJumper-2_P1.3mm_Bridged_RoundedPad1.0x1.5mm -> lib_misc:SolderJumper-3_P1.3mm_Bridged12_RoundedPad1.0x1.5mm
- L1: value Ferrite -> 2.2uH; footprint lib_passives:L_0603 -> lib_passives:WE-XHMI-4030
- L2: value 2.2uH -> Ferrite; footprint lib_passives:WE-XHMI-4030 -> lib_passives:L_0603
- L4: value 6.8nH -> 15nH
- L5: value 15nH -> 6.8nH
- L7: value 1uH -> 6.8uH; footprint lib_passives:WE-XHMI-8080 -> lib_passives:WE-XHMI-1090
- L8: value 6.8uH -> 1uH; footprint lib_passives:WE-XHMI-1510 -> lib_passives:WE-XHMI-8080
- R1: value 47R -> 100R
- R11, R13, R57: value 10K -> 4K7
- R12: value 0R -> 4K7
- R14: value 10K -> 47R
- R15, R16: value 33R -> 41K2
- R17, R18: value 10K -> 41K2
- R19, R21: value 33R -> 10K
- R2: value 100R -> 10K
- R24: value 10K -> 33R
- R25: value 12K1 -> 33R
- R26: value 41K2 -> 10K
- R27, R29: value 41K2 -> 33R
- R28: value 41K2 -> 12K1
- R3, R4: value 4K7 -> 10K
- R35: value 10R -> ~; footprint lib_passives:CRCW0402 -> lib_passives:CRCW0402_QUAD_UART
- R36, R49: value 150R -> 10K
- R38: value 10K -> 150R
- R39: value 150R -> 10R
- R40: value 10R -> 150R
- R41: value 150R -> ~; footprint lib_passives:CRCW0402 -> lib_passives:CRCW0402_QUAD_UART
- R47: value 10K -> ~; footprint lib_passives:CRCW0402 -> lib_passives:CRCW0402_QUAD_UART
- R5: value 4K7 -> 0R
- R50: value 750R -> 150R
- R51: value 267R -> 10R
- R52: value 49R9 -> 150R
- R53: value 100R -> 750R
- R54: value 4K7 -> 267R
- R55: value 4K7 -> 49R9
- R56: value 10K -> 100R
- R58: value 5K1 -> 4K7
- R59, R68: value 5K1 -> 10K
- R60: value 294R -> 10K
- R61: value 2K2 -> 294R
- R62: value 294R -> 8K2
- R63: value 8K2 -> 294R
- R64: value 100R -> 5K1
- R65: value 10K -> 5K1
- R66: value 187K -> 100R
- R67: value 100K -> 2K2
- R69: value 29K4 -> 187K
- R70: value 10R -> 5K1; footprint lib_passives:CRCW2010 -> lib_passives:CRCW0402
- R71: value 10R -> 100K; footprint lib_passives:CRCW2010 -> lib_passives:CRCW0402
- R72: value 10R -> 29K4; footprint lib_passives:CRCW2010 -> lib_passives:CRCW0402
- R73, R75: value 100R -> 10R; footprint lib_passives:CRCW0402 -> lib_passives:CRCW2010
- R74: value 25mR -> 10R; footprint lib_passives:WSR4527 -> lib_passives:CRCW2010
- R77: value 5K1 -> 100R
- R79: value 10M -> 5K1
- R80: value 100K -> 25mR; footprint lib_passives:CRCW0402 -> lib_passives:WSR4527
- R81: value 5k11 -> 100R
- R82: value 499K -> 10M
- R83: value 41K2 -> 150R
- R84: value 53.6k -> 0R; footprint lib_passives:CRCW0402 -> lib_passives:GRT1210
- R85: value 0R -> 25mR; footprint lib_passives:CRCW1210 -> lib_passives:CRCW0805
- R86: value 200K -> 100K
- R87: value 100K -> 53.6k
- R88: value 25mR -> 5k11; footprint lib_passives:CRCW0805 -> lib_passives:CRCW0402
- R89: value 150R -> 41K2
- R90: value 0R -> 150R; footprint lib_passives:GRT1210 -> lib_passives:CRCW0402
- R91: value 150R -> 0R; footprint lib_passives:CRCW0402 -> lib_passives:CRCW1210
- TP28, TP29, TP42, TP43, TP58, TP59, TP86, TP88, TP89: value RCWCTE -> ~; footprint lib_misc:TP_RCW -> lib_misc:TP_2mm
- TP32, TP33, TP48, TP49, TP64, TP65, TP79, TP82, TP84: value ~ -> RCWCTE; footprint lib_misc:TP_2mm -> lib_misc:TP_RCW
- U10, U13: value TXS0108EQWRKSRQ1 -> TPS22996H-Q1; footprint lib_ICs:QFN50P450X250X100-20 -> lib_ICs:SOT583
- U11, U14: value TXS0104VxRUTR -> TXS0108EQWRKSRQ1; footprint lib_ICs:QFN40P170X200X55-12 -> lib_ICs:QFN50P450X250X100-20
- U12, U15, U9: value TPS22996H-Q1 -> TXS0104VxRUTR; footprint lib_ICs:SOT583 -> lib_ICs:QFN40P170X200X55-12
- U7: value TXS0104VxRUTR -> TPS22996H-Q1; footprint lib_ICs:QFN40P170X200X55-12 -> lib_ICs:SOT583
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Connections:
- C1 pad 1: VDD -> /H7_NRST
- C10 pad 1: VDD -> VDDA
- C101 pad 1: /EPS Controller/Battery Charger/PMID -> VSYS
- C103 pad 1: /EPS Controller/Battery Charger/PMID -> VSYS
- C105 pad 1: /EPS Controller/Battery Charger/BAT -> /EPS Controller/Battery Charger/BTST1
- C105 pad 2: CHG- -> /EPS Controller/Battery Charger/SW1
- C106 pad 1: /EPS Controller/Battery Charger/PMID -> /EPS Controller/Battery Charger/BAT
- C106 pad 2: GND -> CHG-
- C107 pad 1: VSYS -> /EPS Controller/Battery Charger/BAT
- C107 pad 2: GND -> CHG-
- C108 pad 1: /EPS Controller/Battery Charger/BAT -> /EPS Controller/Battery Charger/SW2
- C108 pad 2: CHG- -> /EPS Controller/Battery Charger/BTST2
- C109 pad 1: VSYS -> /EPS Controller/Battery Charger/BATP
- C11 pad 1: VDD -> VDDA
- C110 pad 1: VSYS -> /EPS Controller/Battery Charger/REGN
- C115 pad 1: /EPS Controller/Battery Manager/SRP -> Net-(U21-BAT)
- C115 pad 2: /EPS Controller/Battery Manager/SRN -> GND
- C116 pad 1: Net-(U21-BAT) -> /EPS Controller/Battery Manager/REGOUT
- C116 pad 2: GND -> Net-(C116-Pad2)
- C117 pad 1: /EPS Controller/Battery Manager/SRP -> /EPS Controller/Battery Manager/REGSRC
- C117 pad 2: /EPS Controller/Battery Manager/SRN -> Net-(C116-Pad2)
- C118 pad 1: /EPS Controller/Battery Manager/REGSRC -> /EPS Controller/Battery Manager/SRP
- C118 pad 2: Net-(C118-Pad2) -> /EPS Controller/Battery Manager/SRN
- C119 pad 1: /EPS Controller/Battery Manager/REGOUT -> /EPS Controller/Battery Manager/SRP
- C119 pad 2: Net-(C118-Pad2) -> /EPS Controller/Battery Manager/SRN
- C12 pad 1: VDD -> VDD33USB
- C120 pad 1: /EPS Controller/Battery Manager/DSG_S -> CHG+
- C122 pad 1: CHG+ -> /EPS Controller/Battery Manager/DSG_S
- C124 pad 1: VSYS -> /EPS Controller/Voltage Regulators/CBOOT
- C124 pad 2: GND -> /EPS Controller/Voltage Regulators/SW
- C125 pad 1: Net-(U22-VCC) -> VSYS
- C126 pad 1: Net-(U22-EXTCOMP) -> Net-(J30-Pin_2)
- C126 pad 2: AGND -> GND
- C127 pad 1: +3V3 -> Net-(J30-Pin_2)
- C128 pad 1: Net-(C128-Pad1) -> Net-(J30-Pin_2)
- C128 pad 2: AGND -> GND
- C129 pad 1: /EPS Controller/Voltage Regulators/VDDA -> Net-(U22-VCC)
- C129 pad 2: AGND -> GND
- C13 pad 1: VDD -> VDD33USB
- C130 pad 1: /EPS Controller/Voltage Regulators/CBOOT -> /EPS Controller/Voltage Regulators/VDDA
- C130 pad 2: /EPS Controller/Voltage Regulators/SW -> AGND
- C131 pad 1: Net-(J30-Pin_2) -> Net-(U22-EXTCOMP)
- C131 pad 2: GND -> AGND
- C132 pad 1: Net-(J31-Pin_2) -> Net-(C132-Pad1)
- C132 pad 2: GND -> AGND
- C133 pad 1: Net-(J31-Pin_2) -> +3V3
- C15 pad 1: VDD_SMPS_OUT -> VDD
- C16 pad 1: VDDA -> VDD
- C17 pad 1: VDD_SMPS_IN -> VDD
- C18 pad 1: VDDA -> VDD
- C19 pad 1: VCAP -> VDD
- C2 pad 1: VDD -> /EPS Controller/H7_BOOT0
- C2 pad 2: VSS -> Net-(C2-Pad2)
- C20 pad 1: VDD33USB -> VDD
- C21 pad 1: VBAT -> VDD_SMPS_IN
- C22 pad 1: VCAP -> VBAT
- C23 pad 1: VDD33USB -> VDD_SMPS_OUT
- C25 pad 1: /H7_NRST -> VCAP
- C26 pad 1: /EPS Controller/H7_BOOT0 -> VCAP
- C26 pad 2: Net-(C26-Pad2) -> VSS
- C36 pad 1: Net-(U4-VDDCR) -> /Ethernet/3V3_Ethernet
- C38 pad 1: +3V3 -> Net-(U4-VDDCR)
- C39 pad 1: /Ethernet/3V3_Ethernet -> +3V3
- C48 pad 1: /GNSS Card/GPS_SIG_VCCA -> +3V3
- C49 pad 1: /GNSS Card/GPS_GPIO_VCCA -> Net-(U7-VBIAS)
- C50 pad 1: /GNSS Card/GNSS_VDD -> /GNSS Card/GNSS_1V8
- C53 pad 1: +3V3 -> /GNSS Card/GPS_SIG_VCCA
- C54 pad 1: Net-(U9-VBIAS) -> /GNSS Card/GNSS_VDD
- C55 pad 1: /GNSS Card/GNSS_1V8 -> /GNSS Card/GPS_GPIO_VCCA
- C57 pad 1: /LTE Card/LTE_SIG_VCCA -> +3V3
- C58 pad 1: /LTE Card/LTE_GPIO_VCCA -> Net-(U10-VBIAS)
- C59 pad 1: /LTE Card/LTE_VDD -> /LTE Card/LTE_1V8
- C62 pad 1: +3V3 -> /LTE Card/LTE_SIG_VCCA
- C63 pad 1: Net-(U12-VBIAS) -> /LTE Card/LTE_VDD
- C64 pad 1: /LTE Card/LTE_1V8 -> /LTE Card/LTE_GPIO_VCCA
- C66 pad 1: /Auxiliary Card/AUX_SIG_VCCA -> +3V3
- C67 pad 1: /Auxiliary Card/AUX_GPIO_VCCA -> Net-(U13-VBIAS)
- C68 pad 1: /Auxiliary Card/AUX_VDD -> /Auxiliary Card/AUX_1V8
- C71 pad 1: +3V3 -> /Auxiliary Card/AUX_SIG_VCCA
- C72 pad 1: Net-(U15-VBIAS) -> /Auxiliary Card/AUX_VDD
- C73 pad 1: /Auxiliary Card/AUX_1V8 -> /Auxiliary Card/AUX_GPIO_VCCA
- C75 pad 1: /RF Interface/GNSS_RF-IN -> /RF Interface/LNA_RBIAS
- C75 pad 2: /RF Interface/LNA_RF-IN -> VSS
- C76 pad 1: /RF Interface/LNA_RF-GND -> /RF Interface/LNA_RBIAS
- C77 pad 1: /RF Interface/LNA_FB -> /RF Interface/LNA_RBIAS
- C77 pad 2: Net-(C77-Pad2) -> VSS
- C78 pad 1: /RF Interface/LNA_RF-OUT -> /RF Interface/LNA_FB
- C78 pad 2: /RF Interface/RF-SPLIT_SUM -> Net-(C78-Pad2)
- C79 pad 1: /RF Interface/LNA_RBIAS -> /RF Interface/GNSS_RF-IN
- C79 pad 2: VSS -> /RF Interface/LNA_RF-IN
- C80 pad 1: /RF Interface/LNA_RBIAS -> /RF Interface/LNA_RF-OUT
- C80 pad 2: VSS -> /RF Interface/RF-SPLIT_SUM
- C81 pad 1: /RF Interface/LNA_RBIAS -> /RF Interface/LNA_RF-GND
- C91 pad 1: VBUS -> /EPS Controller/Battery Charger/VCHG
- C91 pad 2: AGND -> GND
- C92 pad 1: /EPS Controller/Battery Charger/BTST1 -> /EPS Controller/Battery Charger/VCHG
- C92 pad 2: /EPS Controller/Battery Charger/SW1 -> GND
- C93 pad 1: /EPS Controller/Battery Charger/SW2 -> /EPS Controller/Battery Charger/VCHG
- C93 pad 2: /EPS Controller/Battery Charger/BTST2 -> GND
- C94 pad 1: /EPS Controller/Battery Charger/VCHG -> /EPS Controller/Battery Charger/PMID
- C95 pad 1: /EPS Controller/Battery Charger/VCHG -> /EPS Controller/Battery Charger/PMID
- C96 pad 1: /EPS Controller/Battery Charger/VCHG -> /EPS Controller/Battery Charger/PMID
- C97 pad 1: /EPS Controller/Battery Charger/REGN -> /EPS Controller/Battery Charger/PMID
- C98 pad 1: /EPS Controller/Battery Charger/BATP -> VBUS
- C98 pad 2: GND -> AGND
- C99 pad 1: /EPS Controller/Battery Charger/PMID -> VSYS
- D10 pad 1: /Auxiliary Card/AUX_LED2 -> /Auxiliary Card/AUX_VDD
- D11 pad 1: /Auxiliary Card/AUX_LED1 -> /Auxiliary Card/AUX_LED2
- D12 pad 1: /Auxiliary Card/AUX_VDD -> /Auxiliary Card/AUX_LED1
- D18 pad 1: Net-(D18-Pad1) -> /EPS Controller/Battery Manager/REGSRC
- D19 pad 1: /EPS Controller/Battery Manager/REGSRC -> Net-(D19-Pad1)
- D4 pad 1: /GNSS Card/RTK_STAT -> /GNSS Card/GNSS_VDD
- D5 pad 1: /GNSS Card/GEOFENCE_STAT -> /GNSS Card/RTK_STAT
- D6 pad 1: /GNSS Card/GNSS_VDD -> /GNSS Card/GEOFENCE_STAT
- D7 pad 1: /LTE Card/RTK_STAT -> /LTE Card/LTE_VDD
- D8 pad 1: /LTE Card/GEOFENCE_STAT -> /LTE Card/RTK_STAT
- D9 pad 1: /LTE Card/LTE_VDD -> /LTE Card/GEOFENCE_STAT
- J14 pad 1: /RF Interface/LTE_RF-IN -> /RF Interface/GNSS_CONN1
- J15 pad 1: /RF Interface/AUX_RF-IN -> /RF Interface/GNSS_CONN2
- J16 pad 1: /RF Interface/GNSS_CONN1 -> /RF Interface/LTE_RF-IN
- J17 pad 1: /RF Interface/GNSS_CONN2 -> /RF Interface/AUX_RF-IN
- J18 pad 1: VSS -> +3V3
- J18 pad 2: +3V3 -> /I2C1.SCL
- J18 pad 4: /I2C1.SCL -> VSS
- J19 pad 1: +3V3 -> VSS
- J19 pad 2: /I2C1.SCL -> +3V3
- J19 pad 4: VSS -> /I2C1.SCL
- J28 pad 2: PACK- -> /EPS Controller/Battery Manager/1P
- J29 pad 2: /EPS Controller/Battery Manager/1P -> PACK-
- J30 pad 3: +1V8 -> +3V3
- J31 pad 3: +3V3 -> +1V8
- JP11 pad 1: /EPS Controller/Voltage Regulators/VDDA -> Net-(JP11-Pad1)
- JP11 pad 2: /EPS Controller/Voltage Regulators/PFM -> GND
- JP12 pad 1: Net-(JP12-Pad1) -> /EPS Controller/Voltage Regulators/VDDA
- JP12 pad 2: GND -> /EPS Controller/Voltage Regulators/PFM
- L1 pad 1: VDDA -> VDD_SMPS_OUT
- L1 pad 2: VDD -> VCAP
- L2 pad 1: VDD_SMPS_OUT -> VDDA
- L2 pad 2: VCAP -> VDD
- L4 pad 1: /RF Interface/LNA_RF-IN -> /RF Interface/LNA_RBIAS
- L4 pad 2: /RF Interface/LNA_RF-GND -> /RF Interface/LNA_RF-OUT
- L5 pad 1: /RF Interface/LNA_RBIAS -> /RF Interface/LNA_RF-IN
- L5 pad 2: /RF Interface/LNA_RF-OUT -> /RF Interface/LNA_RF-GND
- L7 pad 1: /EPS Controller/Voltage Regulators/SW_1V8 -> /EPS Controller/Voltage Regulators/SW
- L7 pad 2: Net-(J30-Pin_2) -> /EPS Controller/Voltage Regulators/ISNS+
- L8 pad 1: /EPS Controller/Voltage Regulators/SW -> /EPS Controller/Voltage Regulators/SW_1V8
- L8 pad 2: /EPS Controller/Voltage Regulators/ISNS+ -> Net-(J31-Pin_2)
- Q10 pad 1: /EPS Controller/PG_1V8 -> /EPS Controller/PG_3V3
- Q10 pad 2: Net-(JP12-Pad1) -> Net-(JP11-Pad1)
- Q11 pad 1: /EPS Controller/PG_3V3 -> /EPS Controller/PG_1V8
- Q2 pad 1: Net-(D16-Pad1) -> Net-(D15-Pad1)
- Q2 pad 2: Net-(D16-Pad1) -> Net-(D15-Pad1)
- Q2 pad 3: Net-(D16-Pad1) -> Net-(D15-Pad1)
- Q2 pad 4: Net-(D16-Pad2) -> Net-(D15-Pad2)
- Q2 pad 5: VBUS -> /EPS Controller/Battery Charger/VCHG
- Q2 pad 6: VBUS -> /EPS Controller/Battery Charger/VCHG
- Q2 pad 7: VBUS -> /EPS Controller/Battery Charger/VCHG
- Q2 pad 8: VBUS -> /EPS Controller/Battery Charger/VCHG
- Q2 pad 9: VBUS -> /EPS Controller/Battery Charger/VCHG
- Q3 pad 1: Net-(D15-Pad1) -> Net-(D16-Pad1)
- Q3 pad 2: Net-(D15-Pad1) -> Net-(D16-Pad1)
- Q3 pad 3: Net-(D15-Pad1) -> Net-(D16-Pad1)
- Q3 pad 4: Net-(D15-Pad2) -> Net-(D16-Pad2)
- Q3 pad 5: /EPS Controller/Battery Charger/VCHG -> VBUS
- Q3 pad 6: /EPS Controller/Battery Charger/VCHG -> VBUS
- Q3 pad 7: /EPS Controller/Battery Charger/VCHG -> VBUS
- Q3 pad 8: /EPS Controller/Battery Charger/VCHG -> VBUS
- Q3 pad 9: /EPS Controller/Battery Charger/VCHG -> VBUS
- R1 pad 1: VDDA -> Net-(D1-Pad1)
- R1 pad 2: Net-(U1C-VREF+) -> /STM32H745/H7_LEDBUILTIN
- R10 pad 2: /I2C4.SDA -> /I2C3.SCL
- R11 pad 1: /STM32H745/PDR_ON -> +3V3
- R11 pad 2: +3V3 -> /I2C3.SDA
- R12 pad 1: /STM32H745/PDR_ON -> +3V3
- R12 pad 2: VSS -> /I2C4.SCL
- R13 pad 1: /EPS Controller/H7_BOOT0 -> +3V3
- R13 pad 2: VSS -> /I2C4.SDA
- R14 pad 1: +3V3 -> VDDA
- R14 pad 2: Net-(C26-Pad2) -> Net-(U1C-VREF+)
- R15 pad 1: /Ethernet/RMII.RXD0 -> /Ethernet/3V3_Ethernet
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Other:
- outline, holes or cut-outs redrawn

Commit message: fixed sch
Parts:
- removed D11, D5, D8: LTST-C191TBKT, lib_diodes:LTST-0603
- removed D12, D6, D9: LTST-C191KRKT, lib_diodes:LTST-0603
- removed JP2, JP3, JP5, JP6, JP8, JP9: ~, lib_misc:SolderJumper-2_P1.3mm_Bridged_RoundedPad1.0x1.5mm
- removed R39, R45, R51: 10R, lib_passives:CRCW0402
- removed R40, R46, R52: 150R, lib_passives:CRCW0402
- added NT11: NetTie, lib_misc:NetTie-2_SMD_Pad2.0mm, F.Cu at (188.0, 37.4)
- added kibuzzard-67E082B6: G***, kibuzzard-67E082B6, F.Cu at (225.4, 56.8)
- added kibuzzard-67E082BE: G***, kibuzzard-67E082BE, F.Cu at (221.1, 56.8)
- C105, C108, J27, J28, J29, JP1, JP12, JP4, JP7, R62, R70, R72: moved to B.Cu
- L4, L5: footprint lib_passives:L_0603 -> lib_passives:L_0402
- R80: footprint lib_passives:WSR4527 -> lib_passives:CRCW2512-HP
- moved J17 297.7 mm to (224.5, 125.0)
- moved J16 297.0 mm to (224.5, 107.0)
- moved C79 284.3 mm to (213.0, 136.0), turned to 180 degrees
- moved C81 281.2 mm to (210.8, 133.8), turned to 180 degrees
- moved C78 278.0 mm to (206.6, 134.5), turned to 90 degrees
- moved U16 276.5 mm to (208.8, 135.8), turned to 180 degrees
- moved C77 276.1 mm to (204.6, 132.6)
- moved C75 274.9 mm to (202.5, 133.8), turned to 180 degrees
- moved J15 274.4 mm to (198.0, 139.5)
- moved C76 274.4 mm to (202.5, 132.6), turned to 180 degrees
- moved J14 273.8 mm to (198.0, 130.5), turned to 180 degrees
- moved C80 273.5 mm to (202.4, 136.0), turned to 180 degrees
- moved L5 272.2 mm to (211.3, 135.5), turned to 90 degrees
- moved C82 271.4 mm to (253.7, 59.3)
- moved U18 271.4 mm to (254.9, 55.9)
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Connections:
- J11 pad 16: /Auxiliary Card/AUX_LED2 -> unconnected-(J11-~{LED_2}-Pad16)
- J11 pad 6: /Auxiliary Card/AUX_LED1 -> unconnected-(J11-~{LED_1}-Pad6)
- J5 pad 16: /GNSS Card/RTK_STAT -> unconnected-(J5-~{LED_2}-Pad16)
- J5 pad 6: /GNSS Card/GEOFENCE_STAT -> unconnected-(J5-~{LED_1}-Pad6)
- J8 pad 16: /LTE Card/RTK_STAT -> unconnected-(J8-~{LED_2}-Pad16)
- J8 pad 6: /LTE Card/GEOFENCE_STAT -> unconnected-(J8-~{LED_1}-Pad6)
- NT10 pad 1: CHG- -> CHG+
- NT10 pad 2: GND -> PACK+
- Q5 pad 5: /EPS Controller/Battery Charger/BATP -> CHG+
- Q5 pad 6: /EPS Controller/Battery Charger/BATP -> CHG+
- Q5 pad 7: /EPS Controller/Battery Charger/BATP -> CHG+
- Q5 pad 8: /EPS Controller/Battery Charger/BATP -> CHG+
- Q5 pad 9: /EPS Controller/Battery Charger/BATP -> CHG+
Other:
- board text added: "AUX"
- board text added: "AUX ON"
- board text added: "GNSS"
- board text added: "GNSS ON"
- board text added: "GPIO"
- board text added: "I2C/UART"
- board text added: "I2C/USART"
- board text added: "LTE"
- board text added: "LTE ON"

Commit message: minor changes
Parts:
- added D5: PTVS13VS1UR, lib_diodes:SOD123W, F.Cu at (84.0, 74.2)
- added D6: ESD321DYAR, lib_diodes:SOD523, F.Cu at (84.5, 84.2)
- added D8: ESD321DYAR, lib_diodes:SOD523, F.Cu at (84.5, 86.6)
- added D9: TPD1E05U06-Q1, lib_diodes:SON2P65_100X60X50L50X25N, F.Cu at (85.2, 81.2)
- R80: footprint lib_passives:CRCW2512-HP -> lib_passives:WSL2512-HP
- R84: footprint lib_passives:GRT1210 -> lib_passives:CRCW1210
- moved J1 30.3 mm to (88.5, 61.5)
- moved C98 11.2 mm to (98.7, 78.4)
- moved R73 6.39 mm to (130.8, 72.5)
- moved R74 6.39 mm to (127.2, 72.5)
- moved R75 6.39 mm to (123.8, 72.5)
- moved R68 6.22 mm to (102.5, 76.4)
- moved C111 5.75 mm to (129.0, 76.8)
- moved C112 5.71 mm to (125.5, 76.8)
- moved R61 5.06 mm to (104.8, 72.3)
- moved R63 5.06 mm to (106.0, 72.3)
- moved Q1 4.79 mm to (88.7, 72.4)
- moved C131 4.78 mm to (142.9, 65.4)
- moved C100 4.78 mm to (110.5, 63.6)
- moved C101 4.78 mm to (114.0, 63.6)
- moved C102 4.78 mm to (117.5, 63.6)
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Connections:
- AE1 pad 2: VSS -> /EPS Controller/Battery Charger/SW2
- AE1 pad 3: VSS -> /EPS Controller/Battery Charger/SW2
- AE1 pad 4: VSS -> /EPS Controller/Battery Charger/SW2
- AE1 pad 5: VSS -> /EPS Controller/Battery Charger/SW2
- AE2 pad 2: VSS -> /EPS Controller/Battery Charger/SW2
- AE2 pad 3: VSS -> /EPS Controller/Battery Charger/SW2
- AE2 pad 4: VSS -> /EPS Controller/Battery Charger/SW2
- AE2 pad 5: VSS -> /EPS Controller/Battery Charger/SW2
- AE3 pad 2: VSS -> /EPS Controller/Battery Charger/SW2
- AE3 pad 3: VSS -> /EPS Controller/Battery Charger/SW2
- AE3 pad 4: VSS -> /EPS Controller/Battery Charger/SW2
- AE3 pad 5: VSS -> /EPS Controller/Battery Charger/SW2
- J10 pad 1: VSS -> /EPS Controller/Battery Charger/SW2
- J12 pad 1: VSS -> /EPS Controller/Battery Charger/SW2
- J13 pad 1: VSS -> /EPS Controller/Battery Charger/SW2
- J18 pad 4: VSS -> /EPS Controller/Battery Charger/SW2
- J6 pad 1: VSS -> /EPS Controller/Battery Charger/SW2
- J7 pad 1: VSS -> /EPS Controller/Battery Charger/SW2
- J9 pad 1: VSS -> /EPS Controller/Battery Charger/SW2
Routing:
- net /EPS Controller/Battery Manager/VC5: track 0.00 -> 40.6 mm
- net /EPS Controller/Battery Manager/VC1: track 0.00 -> 34.3 mm
- net /EPS Controller/TS: track 0.00 -> 31.4 mm, vias 0 -> 2
- net /EPS Controller/Battery Manager/VC0: track 0.00 -> 30.5 mm
- net Net-(D15-Pad2): track 0.00 -> 22.6 mm, vias 0 -> 3
- net /EPS Controller/Battery Charger/BATP: track 0.00 -> 21.5 mm, vias 0 -> 2
- net Net-(D16-Pad2): track 0.00 -> 20.9 mm, vias 0 -> 3
- net /EPS Controller/Battery Charger/PVIN: track 0.00 -> 18.1 mm, vias 0 -> 9
- net /EPS Controller/Battery Charger/SDRV: track 0.00 -> 15.8 mm, vias 0 -> 2
- net /EPS Controller/Battery Charger/REGN: track 0.00 -> 12.2 mm, vias 0 -> 2
- net PACK-: track 0.00 -> 8.84 mm, vias 0 -> 1
- net /EPS Controller/Battery Manager/DSG_S: track 0.00 -> 6.83 mm
- net /EPS Controller/BAT_CHG_INT: track 0.00 -> 6.38 mm, vias 0 -> 1
- net /EPS Controller/Battery Charger/SW1: track 0.00 -> 6.19 mm, vias 0 -> 6
- net PACK+: track 0.00 -> 6.14 mm, vias 0 -> 1
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- added copper zone on F.Cu, net /EPS Controller/Battery Charger/BAT
- added copper zone on F.Cu, net /EPS Controller/Battery Charger/PMID
- added copper zone on F.Cu, net /EPS Controller/Battery Charger/PVIN
- added copper zone on B.Cu, net /EPS Controller/Battery Charger/SW1
- added copper zone on F.Cu, net /EPS Controller/Battery Charger/SW1
- added copper zone on In2.Cu, net /EPS Controller/Battery Charger/SW1
- added copper zone on B.Cu, net /EPS Controller/Battery Charger/SW2
- added copper zone on F.Cu, net /EPS Controller/Battery Charger/SW2
- added copper zone on In2.Cu, net /EPS Controller/Battery Charger/SW2
- added copper zone on F.Cu, net /EPS Controller/Battery Charger/VCHG
- added copper zone on F.Cu, net /EPS Controller/Battery Manager/CHG_G
- added copper zone on F.Cu, net /EPS Controller/Battery Manager/DSG_S
- added copper zone on F.Cu, net /EPS Controller/Battery Manager/VC0
- added copper zone on F.Cu, net /EPS Controller/Battery Manager/VC1
- added copper zone on B.Cu, net AGND
- added copper zone on F.Cu, net CHG-
- added copper zone on F.Cu, net GND
- added copper zone on F.Cu, net Net-(D15-Pad1)
- added copper zone on F.Cu, net Net-(D15-Pad2)
- added copper zone on F.Cu, net Net-(D16-Pad1)
- added copper zone on F.Cu, net Net-(D16-Pad2)
- added copper zone on F.Cu, net Net-(Q6-Pad1)
- added copper zone on F.Cu, net PACK-
- added copper zone on In1.Cu, net VSS
- added copper zone on In2.Cu, net VSS
- added copper zone on F.Cu, net VSYS
