File: hardware/electronics/mainBoard/epsController.kicad_sch (KiCad schematic)
At the start: 27 parts, among them SW10 PTS810, SW9 PTS810, U19 STM32L052K8

Commit message: updated ref designators
Parts:
- renumbered R53 to R56, R54 to R57, R55 to R58, R57 to R59, R56 to R60
Changed lines of the file:
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@@
 		(dnp no)
 		(fields_autoplaced yes)
-		(property "Reference" "#PWR0217"
+		(property "Reference" "#PWR0211"
 			(at 185.42 83.82 0)
 			(effects
@@
 			(project "mainBoard"
 				(path "/be16e32f-2ccf-4272-9ec7-94d5fe7a55e0/33ed3f59-5a0e-4fda-9238-d9f0ec67772d"
-					(reference "#PWR0217")
+					(reference "#PWR0211")
 					(unit 1)
 				)
@@
 		(dnp no)
 		(fields_autoplaced yes)
-		(property "Reference" "R55"
+		(property "Reference" "R58"
 			(at 186.69 86.36 0)
 			(do_not_autoplace yes)
@@
 			(project "mainBoard"
 				(path "/be16e32f-2ccf-4272-9ec7-94d5fe7a55e0/33ed3f59-5a0e-4fda-9238-d9f0ec67772d"
-					(reference "R55")
+					(reference "R58")
 					(unit 1)
 				)
@@
 		(dnp no)
 		(fields_autoplaced yes)
-		(property "Reference" "#PWR0220"
+		(property "Reference" "#PWR0213"
 			(at 210.82 125.73 0)
 			(effects
@@
 			(project "mainBoard"
 				(path "/be16e32f-2ccf-4272-9ec7-94d5fe7a55e0/33ed3f59-5a0e-4fda-9238-d9f0ec67772d"
-					(reference "#PWR0220")
+					(reference "#PWR0213")
 					(unit 1)
 				)
@@
 		(dnp no)
 		(fields_autoplaced yes)
-		(property "Reference" "#PWR0211"
+		(property "Reference" "#PWR0205"
 			(at 124.46 53.34 0)
 			(effects
@@
 			(project "mainBoard"
 				(path "/be16e32f-2ccf-4272-9ec7-94d5fe7a55e0/33ed3f59-5a0e-4fda-9238-d9f0ec67772d"
-					(reference "#PWR0211")
+					(reference "#PWR0205")
 					(unit 1)
 				)
@@
 		(dnp no)
 		(fields_autoplaced yes)
-		(property "Reference" "R57"
+		(property "Reference" "R59"
 			(at 212.09 125.73 0)
 			(do_not_autoplace yes)
@@
 			(project "mainBoard"
 				(path "/be16e32f-2ccf-4272-9ec7-94d5fe7a55e0/33ed3f59-5a0e-4fda-9238-d9f0ec67772d"
-					(reference "R57")
+					(reference "R59")
 					(unit 1)
 				)
@@
 		(dnp no)
 		(fields_autoplaced yes)
-		(property "Reference" "#PWR0205"
+		(property "Reference" "#PWR0219"
 			(at 30.48 184.15 0)
 			(effects
@@
 			(project "mainBoard"
 				(path "/be16e32f-2ccf-4272-9ec7-94d5fe7a55e0/33ed3f59-5a0e-4fda-9238-d9f0ec67772d"
-					(reference "#PWR0205")
+					(reference "#PWR0219")
 					(unit 1)
 				)
@@
 		(dnp no)
 		(fields_autoplaced yes)
-		(property "Reference" "#PWR0206"
+		(property "Reference" "#PWR0220"
 			(at 30.48 191.77 0)
 			(effects
@@
 			(project "mainBoard"
 				(path "/be16e32f-2ccf-4272-9ec7-94d5fe7a55e0/33ed3f59-5a0e-4fda-9238-d9f0ec67772d"
-					(reference "#PWR0206")
+					(reference "#PWR0220")
 					(unit 1)
 				)
@@
 		(dnp no)
 		(fields_autoplaced yes)
-		(property "Reference" "#PWR0218"
+		(property "Reference" "#PWR0216"
 			(at 195.58 156.21 0)
 			(effects
@@
 			(project "mainBoard"
 				(path "/be16e32f-2ccf-4272-9ec7-94d5fe7a55e0/33ed3f59-5a0e-4fda-9238-d9f0ec67772d"
-					(reference "#PWR0218")
+					(reference "#PWR0216")
 					(unit 1)
 				)
@@
 		(dnp no)
 		(fields_autoplaced yes)
-		(property "Reference" "#PWR0214"
+		(property "Reference" "#PWR0217"
 			(at 139.7 157.48 0)
 			(effects
@@
 			(project "mainBoard"
 				(path "/be16e32f-2ccf-4272-9ec7-94d5fe7a55e0/33ed3f59-5a0e-4fda-9238-d9f0ec67772d"
-					(reference "#PWR0214")
+					(reference "#PWR0217")
 					(unit 1)
 				)
@@
 		(dnp no)
 		(fields_autoplaced yes)
-		(property "Reference" "#PWR0213"
+		(property "Reference" "#PWR0207"
 			(at 139.7 60.96 0)
 			(effects
@@
 			(project "mainBoard"
 				(path "/be16e32f-2ccf-4272-9ec7-94d5fe7a55e0/33ed3f59-5a0e-4fda-9238-d9f0ec67772d"
-					(reference "#PWR0213")
+					(reference "#PWR0207")
 					(unit 1)
 				)
@@
 		(dnp no)
 		(fields_autoplaced yes)
-		(property "Reference" "#PWR0204"
+		(property "Reference" "#PWR0218"
 			(at 30.48 176.53 0)
 			(effects
@@
 			(project "mainBoard"
 				(path "/be16e32f-2ccf-4272-9ec7-94d5fe7a55e0/33ed3f59-5a0e-4fda-9238-d9f0ec67772d"
-					(reference "#PWR0204")
+					(reference "#PWR0218")
 					(unit 1)
 				)
@@
 		(dnp no)
 		(fields_autoplaced yes)
-		(property "Reference" "#PWR0210"
+		(property "Reference" "#PWR0204"
 			(at 124.46 41.91 0)
 			(effects
@@
 			(project "mainBoard"
 				(path "/be16e32f-2ccf-4272-9ec7-94d5fe7a55e0/33ed3f59-5a0e-4fda-9238-d9f0ec67772d"
-					(reference "#PWR0210")
+					(reference "#PWR0204")
 					(unit 1)
 				)
@@
 		(dnp no)
 		(fields_autoplaced yes)
-		(property "Reference" "#PWR0212"
+		(property "Reference" "#PWR0206"
 			(at 134.62 60.96 0)
 			(effects
@@
 			(project "mainBoard"
 				(path "/be16e32f-2ccf-4272-9ec7-94d5fe7a55e0/33ed3f59-5a0e-4fda-9238-d9f0ec67772d"
-					(reference "#PWR0212")
+					(reference "#PWR0206")
 					(unit 1)
 				)
@@
 		(dnp no)
 		(fields_autoplaced yes)
-		(property "Reference" "#PWR0208"
+		(property "Reference" "#PWR0215"
 			(at 76.2 149.86 0)
 			(effects
@@
 			(project "mainBoard"
 				(path "/be16e32f-2ccf-4272-9ec7-94d5fe7a55e0/33ed3f59-5a0e-4fda-9238-d9f0ec67772d"
-					(reference "#PWR0208")
+					(reference "#PWR0215")
 					(unit 1)
 				)
@@
 		(dnp no)
 		(fields_autoplaced yes)
-		(property "Reference" "#PWR0219"
+		(property "Reference" "#PWR0212"
 			(at 210.82 115.57 0)
 			(effects
@@
 			(project "mainBoard"
 				(path "/be16e32f-2ccf-4272-9ec7-94d5fe7a55e0/33ed3f59-5a0e-4fda-9238-d9f0ec67772d"
-					(reference "#PWR0219")
+					(reference "#PWR0212")
 					(unit 1)
 				)
@@
 		(dnp no)
 		(fields_autoplaced yes)
-		(property "Reference" "R56"
+		(property "Reference" "R60"
 			(at 196.85 148.59 0)
 			(do_not_autoplace yes)
@@
 			(project "mainBoard"
 				(path "/be16e32f-2ccf-4272-9ec7-94d5fe7a55e0/33ed3f59-5a0e-4fda-9238-d9f0ec67772d"
-					(reference "R56")
+					(reference "R60")
 					(unit 1)
 				)
@@
 		(dnp no)
 		(fields_autoplaced yes)
-		(property "Reference" "R53"
+		(property "Reference" "R56"
 			(at 101.6 68.58 0)
 			(do_not_autoplace yes)
@@
 			(project "mainBoard"
 				(path "/be16e32f-2ccf-4272-9ec7-94d5fe7a55e0/33ed3f59-5a0e-4fda-9238-d9f0ec67772d"
-					(reference "R53")
+					(reference "R56")
 					(unit 1)
 				)
@@
 		(dnp no)
 		(fields_autoplaced yes)
-		(property "Reference" "R54"
+		(property "Reference" "R57"
 			(at 177.8 86.36 0)
 			(do_not_autoplace yes)
@@
 			(project "mainBoard"
 				(path "/be16e32f-2ccf-4272-9ec7-94d5fe7a55e0/33ed3f59-5a0e-4fda-9238-d9f0ec67772d"
-					(reference "R54")
+					(reference "R57")
 					(unit 1)
 				)
@@
 		(dnp no)
 		(fields_autoplaced yes)
-		(property "Reference" "#PWR0207"
+		(property "Reference" "#PWR0214"
 			(at 76.2 134.62 0)
 			(effects
@@
 			(project "mainBoard"
 				(path "/be16e32f-2ccf-4272-9ec7-94d5fe7a55e0/33ed3f59-5a0e-4fda-9238-d9f0ec67772d"
-					(reference "#PWR0207")
+					(reference "#PWR0214")
 					(unit 1)
 				)
@@
 		(dnp no)
 		(fields_autoplaced yes)
-		(property "Reference" "#PWR0215"
+		(property "Reference" "#PWR0208"
 			(at 144.78 60.96 0)
 			(effects
@@
 			(project "mainBoard"
 				(path "/be16e32f-2ccf-4272-9ec7-94d5fe7a55e0/33ed3f59-5a0e-4fda-9238-d9f0ec67772d"
-					(reference "#PWR0215")
+					(reference "#PWR0208")
 					(unit 1)
 				)
@@
 		(dnp no)
 		(fields_autoplaced yes)
-		(property "Reference" "#PWR0216"
+		(property "Reference" "#PWR0210"
 			(at 176.53 83.82 0)
 			(effects
@@
 			(project "mainBoard"
 				(path "/be16e32f-2ccf-4272-9ec7-94d5fe7a55e0/33ed3f59-5a0e-4fda-9238-d9f0ec67772d"
-					(reference "#PWR0216")
+					(reference "#PWR0210")
 					(unit 1)
 				)

Commit message: redefined symbol refs
Parts:
- added C88: 100nF, lib_passives:GCM0402, symbol lib_sch:C
- renumbered C88 to C89, C89 to C90, D13 to D7, D14 to D8, R56 to R50, R57 to R51, R58 to R52, R59 to R53, R60 to R54
Connections:
- net +3V3: now also C88.1
- net VSS: now also C88.2
