File: hardware/electronics/mainBoard/voltageRegulators.kicad_sch (KiCad schematic)
At the start: 44 parts, among them J30 Conn_01x04_Pin, J31 Conn_01x04_Pin, Q10 BSS138-7-F, Q11 BSS138-7-F, Q8 CSD17581Q3A, Q9 CSD17581Q3A, U22 LM25148-Q1, U23 TPS62A01

Commit message: updated sheet date
Parts:
- J30, J31: footprint lib_connectors:conn_01x04_254_right_angle -> lib_connectors:conn_01x04_254; DKPN S1111EC-04-ND -> S1011EC-04-ND; MPN PRPC004SBAN-M71RC -> PRPC004SAAN-RC
Changed lines of the file:
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@@
 	(title_block
 		(title "Voltage Regulators")
-		(date "2025-03-20")
+		(date "2025-03-31")
 		(rev "1")
 		(comment 2 "PROTOTYPE")
@@
 			)
 		)
-		(property "Footprint" "lib_connectors:conn_01x04_254_right_angle"
+		(property "Footprint" "lib_connectors:conn_01x04_254"
 			(at 241.3 35.56 0)
 			(effects
@@
 			)
 		)
-		(property "Datasheet" "datasheets/Sullins-xRxCzzzSxxN-M71RC.pdf"
+		(property "Datasheet" "datasheets/Sullins-xRxCzzzSxxN-RC.pdf"
 			(at 241.3 35.56 0)
 			(effects
@@
 			)
 		)
-		(property "Description" "CONN HEADER R/A 4POS 2.54MM"
+		(property "Description" "CONN HEADER VERT 4POS 2.54MM"
 			(at 241.3 35.56 0)
 			(effects
@@
 			)
 		)
-		(property "MPN" "PRPC004SBAN-M71RC"
+		(property "MPN" "PRPC004SAAN-RC"
 			(at 241.3 35.56 0)
 			(effects
@@
 			)
 		)
-		(property "DKPN" "S1111EC-04-ND"
+		(property "DKPN" "S1011EC-04-ND"
 			(at 241.3 35.56 0)
 			(effects
@@
 	)
 	(symbol
+		(lib_id "lib_sch:Conn_01x04_Pin")
+		(at 187.96 124.46 180)
+		(unit 1)
+		(exclude_from_sim no)
+		(in_bom yes)
+		(on_board yes)
+		(dnp no)
+		(property "Reference" "J31"
+			(at 187.96 114.3 0)
+			(effects
+				(font
+					(size 1.27 1.27)
+				)
+			)
+		)
+		(property "Value" "Conn_01x04_Pin"
+			(at 187.96 116.84 0)
+			(effects
+				(font
+					(size 1.27 1.27)
+				)
+			)
+		)
+		(property "Footprint" "lib_connectors:conn_01x04_254"
+			(at 187.96 124.46 0)
+			(effects
+				(font
+					(size 1.27 1.27)
+				)
+				(hide yes)
+			)
+		)
+		(property "Datasheet" "datasheets/Sullins-xRxCzzzSxxN-RC.pdf"
+			(at 187.96 124.46 0)
+			(effects
+				(font
+					(size 1.27 1.27)
+				)
+				(hide yes)
+			)
+		)
+		(property "Description" "CONN HEADER VERT 4POS 2.54MM"
+			(at 187.96 124.46 0)
+			(effects
+				(font
+					(size 1.27 1.27)
+				)
+				(hide yes)
+			)
+		)
+		(property "Manufacturer" "Sullins Connector Solutions"
+			(at 187.96 124.46 0)
+			(effects
+				(font
+					(size 1.27 1.27)
+				)
+				(hide yes)
+			)
+		)
+		(property "MPN" "PRPC004SAAN-RC"
+			(at 187.96 124.46 0)
+			(effects
+				(font
+					(size 1.27 1.27)
+				)
+				(hide yes)
+			)
+		)
+		(property "DKPN" "S1011EC-04-ND"
+			(at 187.96 124.46 0)
+			(effects
+				(font
+					(size 1.27 1.27)
+				)
+				(hide yes)
+			)
+		)
+		(pin "1"
+		)
+		(pin "2"
+		)
+		(pin "3"
+		)
+		(pin "4"
+		)
+		(instances
+			(project "mainBoard"
+				(path "/be16e32f-2ccf-4272-9ec7-94d5fe7a55e0/33ed3f59-5a0e-4fda-9238-d9f0ec67772d/8fe11cde-b323-4b38-a163-6c6134ab47c7"
+					(reference "J31")
+					(unit 1)
+				)
+			)
+		)
+	)
+	(symbol
 		(lib_id "lib_sch:NMOS_SGD_PWR")
 		(at 177.8 38.1 270)
@@
 					(unit 1)
 				)
-			)
-		)
-	)
-	(symbol
-		(lib_id "lib_sch:Conn_01x04_Pin")
-		(at 187.96 124.46 180)
-		(unit 1)
-		(exclude_from_sim no)
-		(in_bom yes)
-		(on_board yes)
-		(dnp no)
-		(property "Reference" "J31"
-			(at 187.96 114.3 0)
-			(effects
-				(font
-					(size 1.27 1.27)
-				)
-			)
-		)
-		(property "Value" "Conn_01x04_Pin"
-			(at 187.96 116.84 0)
-			(effects
-				(font
-					(size 1.27 1.27)
-				)
-			)
-		)
-		(property "Footprint" "lib_connectors:conn_01x04_254_right_angle"
-			(at 187.96 124.46 0)
-			(effects
-				(font
-					(size 1.27 1.27)
-				)
-				(hide yes)
-			)
-		)
-		(property "Datasheet" "datasheets/Sullins-xRxCzzzSxxN-M71RC.pdf"
-			(at 187.96 124.46 0)
-			(effects
-				(font
-					(size 1.27 1.27)
-				)
-				(hide yes)
-			)
-		)
-		(property "Description" "CONN HEADER R/A 4POS 2.54MM"
-			(at 187.96 124.46 0)
-			(effects
-				(font
-					(size 1.27 1.27)
-				)
-				(hide yes)
-			)
-		)
-		(property "Manufacturer" "Sullins Connector Solutions"
-			(at 187.96 124.46 0)
-			(effects
-				(font
-					(size 1.27 1.27)
-				)
-				(hide yes)
-			)
-		)
-		(property "MPN" "PRPC004SBAN-M71RC"
-			(at 187.96 124.46 0)
-			(effects
-				(font
-					(size 1.27 1.27)
-				)
-				(hide yes)
-			)
-		)
-		(property "DKPN" "S1111EC-04-ND"
-			(at 187.96 124.46 0)
-			(effects
-				(font
-					(size 1.27 1.27)
-				)
-				(hide yes)
-			)
-		)
-		(pin "1"
-		)
-		(pin "2"
-		)
-		(pin "3"
-		)
-		(pin "4"
-		)
-		(instances
-			(project "mainBoard"
-				(path "/be16e32f-2ccf-4272-9ec7-94d5fe7a55e0/33ed3f59-5a0e-4fda-9238-d9f0ec67772d/8fe11cde-b323-4b38-a163-6c6134ab47c7"
-					(reference "J31")
-					(unit 1)
-				)

Commit message: redefined symbol refs
Parts:
- renumbered C124 to C125, C125 to C126, C126 to C127, C127 to C128, C128 to C129, C129 to C130, C130 to C131, C131 to C132, C132 to C133, C133 to C134, C134 to C135, D21 to D19, D22 to D20, JP11 to JP5, JP12 to JP6, JP13 to JP7, R83 to R77, R84 to R78, R85 to R79, R86 to R80, R87 to R81, R88 to R82, R89 to R83, R90 to R84, R91 to R85, R92 to R86, R93 to R87, R94 to R88
