File: hardware/electronics/mainBoard/debugger_l0.kicad_sch (KiCad schematic)
At the start: 21 parts, among them J23 STEMMA-QT, J33 USB_B, SW13 PTS810, SW14 PTS810, U32 AP2112K-3.3, U33 STM32F103TBU6

Commit message: debugger stuff
Connections:
- net Debug_8MHz renamed L0_Debug_8MHz
- net L0_NRST renamed L0_nRST
- net UART1_RX renamed L0_DBG_RX
- net UART1_TX renamed L0_DBG_TX
- no-connect marks 14 -> 15
Other:
- moved on the sheet: R106, R107
Changed lines of the file:
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@@
 	)
 	(no_connect
+		(at 124.46 74.93)
+	)
+	(no_connect
 		(at 251.46 152.4)
 	)
@@
 	(wire
 		(pts
-			(xy 109.22 99.06) (xy 109.22 100.33)
+			(xy 93.98 99.06) (xy 93.98 100.33)
 		)
 		(stroke
@@
 	(wire
 		(pts
-			(xy 92.71 99.06) (xy 101.6 99.06)
+			(xy 77.47 99.06) (xy 86.36 99.06)
 		)
 		(stroke
@@
 	(wire
 		(pts
-			(xy 109.22 104.14) (xy 109.22 102.87)
+			(xy 93.98 104.14) (xy 93.98 102.87)
 		)
 		(stroke
@@
 	(wire
 		(pts
-			(xy 109.22 102.87) (xy 124.46 102.87)
+			(xy 93.98 102.87) (xy 124.46 102.87)
 		)
 		(stroke
@@
 	(wire
 		(pts
-			(xy 106.68 99.06) (xy 109.22 99.06)
+			(xy 91.44 99.06) (xy 93.98 99.06)
 		)
 		(stroke
@@
 	(wire
 		(pts
-			(xy 92.71 104.14) (xy 101.6 104.14)
+			(xy 77.47 104.14) (xy 86.36 104.14)
 		)
 		(stroke
@@
 	(wire
 		(pts
-			(xy 106.68 104.14) (xy 109.22 104.14)
+			(xy 91.44 104.14) (xy 93.98 104.14)
 		)
 		(stroke
@@
 	(wire
 		(pts
-			(xy 109.22 100.33) (xy 124.46 100.33)
+			(xy 93.98 100.33) (xy 124.46 100.33)
 		)
 		(stroke
@@
 	)
 	(label "USB_D_N"
-		(at 92.71 99.06 0)
+		(at 77.47 99.06 0)
 		(effects
 			(font
@@
 	)
 	(label "USB_D_P"
-		(at 92.71 104.14 0)
+		(at 77.47 104.14 0)
 		(effects
 			(font
@@
 		)
 	)
+	(hierarchical_label "L0_DBG_RX"
+		(shape input)
+		(at 111.76 97.79 180)
+		(effects
+			(font
+				(size 1.27 1.27)
+			)
+			(justify right)
+		)
+	)
 	(hierarchical_label "L0_SWDIO"
 		(shape bidirectional)
@@
 		)
 	)
-	(hierarchical_label "Debug_8MHz"
+	(hierarchical_label "L0_Debug_8MHz"
 		(shape input)
 		(at 165.1 92.71 0)
@@
 		)
 	)
-	(hierarchical_label "L0_NRST"
+	(hierarchical_label "L0_nRST"
 		(shape output)
 		(at 111.76 69.85 180)
@@
 		)
 	)
+	(hierarchical_label "L0_DBG_TX"
+		(shape output)
+		(at 111.76 95.25 180)
+		(effects
+			(font
+				(size 1.27 1.27)
+			)
+			(justify right)
+		)
+	)
 	(symbol
 		(lib_id "lib_sch:R")
@@
 	(symbol
 		(lib_id "lib_sch:R_horizontal")
-		(at 104.14 104.14 0)
+		(at 88.9 104.14 0)
 		(unit 1)
 		(exclude_from_sim no)
@@
 		(dnp no)
 		(property "Reference" "R107"
-			(at 104.14 102.87 0)
+			(at 88.9 102.87 0)
 			(do_not_autoplace yes)
 			(effects
@@
 		)
 		(property "Value" "22R"
-			(at 104.14 105.41 0)
+			(at 88.9 105.41 0)
 			(do_not_autoplace yes)
 			(effects
@@
 		)
 		(property "Footprint" "lib_passives:CRCW0402"
-			(at 101.6 104.14 90)
+			(at 86.36 104.14 90)
 			(effects
 				(font
@@
 		)
 		(property "Datasheet" "datasheets/Vishay-Dale-DCRCWe3.pdf"
-			(at 101.6 104.14 90)
+			(at 86.36 104.14 90)
 			(effects
 				(font
@@
 		)
 		(property "Description" "RES SMD 22 OHM 1% 1/16W 0402"
-			(at 104.14 104.14 0)
+			(at 88.9 104.14 0)
 			(effects
 				(font
@@
 		)
 		(property "Manufacturer" "Vishay Dale"
-			(at 101.6 104.14 90)
+			(at 86.36 104.14 90)
 			(effects
 				(font
@@
 		)
 		(property "MPN" "CRCW040222R0FKED"
-			(at 101.6 104.14 90)
+			(at 86.36 104.14 90)
 			(effects
 				(font
@@
 		)
 		(property "DKPN" "541-22.0LCT-ND"
-			(at 104.14 104.14 0)
+			(at 88.9 104.14 0)
 			(effects
 				(font
@@
 		)
 		(property "Tolerance" "1%"
-			(at 104.14 106.68 0)
+			(at 88.9 106.68 0)
 			(do_not_autoplace yes)
 			(effects
@@
 		)
 		(property "Power Rating" "62m5W"
-			(at 104.14 105.41 0)
+			(at 88.9 105.41 0)
 			(do_not_autoplace yes)
 			(effects
@@
 		)
 		(property "Package" "0402"
-			(at 104.14 106.68 0)
+			(at 88.9 106.68 0)
 			(do_not_autoplace yes)
 			(effects
@@
 	(symbol
 		(lib_id "lib_sch:R_horizontal")
-		(at 104.14 99.06 0)
+		(at 88.9 99.06 0)
 		(unit 1)
 		(exclude_from_sim no)
@@
 		(dnp no)
 		(property "Reference" "R106"
-			(at 104.14 97.79 0)
+			(at 88.9 97.79 0)
 			(do_not_autoplace yes)
 			(effects
@@
 		)
 		(property "Value" "22R"
-			(at 104.14 100.33 0)
+			(at 88.9 100.33 0)
 			(do_not_autoplace yes)
 			(effects
@@
 		)
 		(property "Footprint" "lib_passives:CRCW0402"
-			(at 101.6 99.06 90)
+			(at 86.36 99.06 90)
 			(effects
 				(font
@@
 		)
 		(property "Datasheet" "datasheets/Vishay-Dale-DCRCWe3.pdf"
-			(at 101.6 99.06 90)
+			(at 86.36 99.06 90)
 			(effects
 				(font
@@
 		)
 		(property "Description" "RES SMD 22 OHM 1% 1/16W 0402"
-			(at 104.14 99.06 0)
+			(at 88.9 99.06 0)
 			(effects
 				(font
@@
 		)
 		(property "Manufacturer" "Vishay Dale"
-			(at 101.6 99.06 90)
+			(at 86.36 99.06 90)
 			(effects
 				(font
@@
 		)
 		(property "MPN" "CRCW040222R0FKED"
-			(at 101.6 99.06 90)
+			(at 86.36 99.06 90)
 			(effects
 				(font
@@
 		)
 		(property "DKPN" "541-22.0LCT-ND"
-			(at 104.14 99.06 0)
+			(at 88.9 99.06 0)
 			(effects
 				(font
@@
 		)
 		(property "Tolerance" "1%"
-			(at 104.14 101.6 0)
+			(at 88.9 101.6 0)
 			(do_not_autoplace yes)
 			(effects
@@
 		)
 		(property "Power Rating" "62m5W"
-			(at 104.14 100.33 0)
+			(at 88.9 100.33 0)
 			(do_not_autoplace yes)
 			(effects
@@
 		)
 		(property "Package" "0402"
-			(at 104.14 101.6 0)
+			(at 88.9 101.6 0)
 			(do_not_autoplace yes)
 			(effects
