File: hardware/electronics/mainBoard/usb_hub.kicad_sch (KiCad schematic)
At the start: 23 parts, among them J9 MUSBRM1C1M0, U4 USB2422-I/MJ

Commit message: fixed file names
Other:
- title: Awohali USB Hub -> Awohali - USB Hub
Changed lines of the file:
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@@
 	(paper "B")
 	(title_block
-		(title "Awohali USB Hub")
+		(title "Awohali - USB Hub")
 		(date "2025-07-01")
 		(rev "1")
