File: hardware/electronics/bms_breakout/battery_charger.kicad_sch (KiCad schematic)
At the start: 35 parts, among them J5 VAL, J6 VAL, Q1 BUK961R6, U1 BQ25798

Commit message: added footprints for all resistors and capacitors
Parts:
- C1, C12, C13, C14, C15, C16, C17, C18, C2, C5, C6, C7: footprint (none) -> DS-Capacitors-SMD:MLCC1206
- C10: footprint (none) -> 12065C475K4T4A
- C11, C19, C3, C4, C8, C9: footprint (none) -> DS-Capacitors-SMD:MLCC0603
- R1, R2, R3, R4, R5, R6, R7, R8: footprint (none) -> DS-Resistors-SMD:CRCW0603
Changed lines of the file:
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@@
 			)
 		)
-		(property "Footprint" ""
+		(property "Footprint" "DS-Capacitors-SMD:MLCC0603"
 			(at 142.24 80.645 0)
 			(effects
@@
 			)
 		)
-		(property "Footprint" ""
+		(property "Footprint" "DS-Capacitors-SMD:MLCC0603"
 			(at 87.63 81.915 0)
 			(effects
@@
 			)
 		)
-		(property "Footprint" ""
+		(property "Footprint" "DS-Capacitors-SMD:MLCC1206"
 			(at 173.99 108.585 0)
 			(effects
@@
 			)
 		)
-		(property "Footprint" ""
+		(property "Footprint" "DS-Capacitors-SMD:MLCC0603"
 			(at 92.71 104.775 0)
 			(effects
@@
 			)
 		)
-		(property "Footprint" ""
+		(property "Footprint" "DS-Capacitors-SMD:MLCC1206"
 			(at 162.56 98.425 0)
 			(effects
@@
 			)
 		)
-		(property "Footprint" ""
+		(property "Footprint" "DS-Resistors-SMD:CRCW0603"
 			(at 207.01 93.98 0)
 			(effects
@@
 			)
 		)
-		(property "Footprint" ""
+		(property "Footprint" "DS-Capacitors-SMD:MLCC1206"
 			(at 80.01 81.915 0)
 			(effects
@@
 			)
 		)
-		(property "Footprint" ""
+		(property "Footprint" "DS-Resistors-SMD:CRCW0603"
 			(at 73.66 134.62 0)
 			(effects
@@
 			)
 		)
-		(property "Footprint" ""
+		(property "Footprint" "DS-Capacitors-SMD:MLCC0603"
 			(at 139.7 98.425 0)
 			(effects
@@
 			)
 		)
-		(property "Footprint" ""
+		(property "Footprint" "DS-Capacitors-SMD:MLCC1206"
 			(at 165.1 80.645 0)
 			(effects
@@
 			)
 		)
-		(property "Footprint" ""
+		(property "Footprint" "DS-Resistors-SMD:CRCW0603"
 			(at 190.5 93.98 0)
 			(effects
@@
 			)
 		)
-		(property "Footprint" ""
+		(property "Footprint" "DS-Capacitors-SMD:MLCC1206"
 			(at 177.8 98.425 0)
 			(effects
@@
 			)
 		)
-		(property "Footprint" ""
+		(property "Footprint" "DS-Resistors-SMD:CRCW0603"
 			(at 142.24 116.84 90)
 			(effects
@@
 			)
 		)
-		(property "Footprint" ""
+		(property "Footprint" "DS-Capacitors-SMD:MLCC1206"
 			(at 149.86 80.645 0)
 			(effects
@@
 			)
 		)
-		(property "Footprint" ""
+		(property "Footprint" "DS-Resistors-SMD:CRCW0603"
 			(at 132.08 86.36 90)
 			(effects
@@
 			)
 		)
-		(property "Footprint" ""
+		(property "Footprint" "DS-Capacitors-SMD:MLCC0603"
 			(at 135.89 118.745 0)
 			(effects
@@
 			)
 		)
-		(property "Footprint" ""
+		(property "Footprint" "DS-Capacitors-SMD:MLCC1206"
 			(at 157.48 80.645 0)
 			(effects
@@
 			)
 		)
-		(property "Footprint" ""
+		(property "Footprint" "DS-Capacitors-SMD:MLCC1206"
 			(at 147.32 98.425 0)
 			(effects
@@
 			)
 		)
-		(property "Footprint" ""
+		(property "Footprint" "DS-Capacitors-SMD:MLCC0603"
 			(at 92.71 120.015 0)
 			(effects
@@
 			)
 		)
-		(property "Footprint" ""
+		(property "Footprint" "DS-Capacitors-SMD:MLCC1206"
 			(at 154.94 98.425 0)
 			(effects
@@
 			)
 		)
-		(property "Footprint" ""
+		(property "Footprint" "DS-Capacitors-SMD:MLCC1206"
 			(at 166.37 108.585 0)
 			(effects
@@
 			)
 		)
-		(property "Footprint" ""
+		(property "Footprint" "DS-Resistors-SMD:CRCW0603"
 			(at 82.55 130.81 90)
 			(effects
@@
 			)
 		)
-		(property "Footprint" ""
+		(property "Footprint" "DS-Resistors-SMD:CRCW0603"
 			(at 190.5 81.28 0)
 			(effects
@@
 			)
 		)
-		(property "Footprint" ""
+		(property "Footprint" "12065C475K4T4A"
 			(at 88.9 120.015 0)
 			(effects
@@
 			)
 		)
-		(property "Footprint" ""
+		(property "Footprint" "DS-Capacitors-SMD:MLCC1206"
 			(at 72.39 81.915 0)
 			(effects
@@
 			)
 		)
-		(property "Footprint" ""
+		(property "Footprint" "DS-Resistors-SMD:CRCW0603"
 			(at 207.01 81.28 0)
 			(effects
@@
 			)
 		)
-		(property "Footprint" ""
+		(property "Footprint" "DS-Capacitors-SMD:MLCC1206"
 			(at 170.18 98.425 0)
 			(effects
