File: hardware/electronics/bms_breakout/battery_monitor.kicad_sch (KiCad schematic)
At the start: 31 parts, among them Q2 CSD18532Q5B, Q3 CSD18532Q5B, U2 BQ76905

Commit message: added footprints for all resistors and capacitors
Parts:
- C20, C21, C23: footprint (none) -> DS-Capacitors-SMD:MLCC0805
- C22, C24, C25, C26, C27, C28, C29, C30: footprint (none) -> DS-Capacitors-SMD:MLCC0603
- R10, R11, R12, R13, R15, R16, R17, R18, R9: footprint (none) -> DS-Resistors-SMD:CRCW0603
- R14: footprint (none) -> DS-Resistors-SMD:WSLHP2010
Changed lines of the file:
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@@
 			)
 		)
-		(property "Footprint" ""
+		(property "Footprint" "DS-Resistors-SMD:CRCW0603"
 			(at 190.5 110.49 0)
 			(effects
@@
 			)
 		)
-		(property "Footprint" ""
+		(property "Footprint" "DS-Capacitors-SMD:MLCC0603"
 			(at 190.5 142.875 0)
 			(effects
@@
 			)
 		)
-		(property "Footprint" ""
+		(property "Footprint" "DS-Capacitors-SMD:MLCC0603"
 			(at 134.62 90.805 0)
 			(effects
@@
 			)
 		)
-		(property "Footprint" ""
+		(property "Footprint" "DS-Resistors-SMD:CRCW0603"
 			(at 147.32 118.11 90)
 			(effects
@@
 			)
 		)
-		(property "Footprint" ""
+		(property "Footprint" "DS-Capacitors-SMD:MLCC0805"
 			(at 142.24 90.805 0)
 			(effects
@@
 			)
 		)
-		(property "Footprint" ""
+		(property "Footprint" "DS-Resistors-SMD:WSLHP2010"
 			(at 156.21 119.38 0)
 			(effects
@@
 			)
 		)
-		(property "Footprint" ""
+		(property "Footprint" "DS-Capacitors-SMD:MLCC0603"
 			(at 130.81 120.015 0)
 			(effects
@@
 			)
 		)
-		(property "Footprint" ""
+		(property "Footprint" "DS-Resistors-SMD:CRCW0603"
 			(at 148.59 88.9 90)
 			(effects
@@
 			)
 		)
-		(property "Footprint" ""
+		(property "Footprint" "DS-Capacitors-SMD:MLCC0603"
 			(at 177.8 142.875 0)
 			(effects
@@
 			)
 		)
-		(property "Footprint" ""
+		(property "Footprint" "DS-Resistors-SMD:CRCW0603"
 			(at 88.9 119.38 0)
 			(effects
@@
 			)
 		)
-		(property "Footprint" ""
+		(property "Footprint" "DS-Capacitors-SMD:MLCC0603"
 			(at 46.99 52.705 0)
 			(effects
@@
 			)
 		)
-		(property "Footprint" ""
+		(property "Footprint" "DS-Resistors-SMD:CRCW0603"
 			(at 147.32 125.73 90)
 			(effects
@@
 			)
 		)
-		(property "Footprint" ""
+		(property "Footprint" "DS-Capacitors-SMD:MLCC0805"
 			(at 91.44 102.235 0)
 			(effects
@@
 			)
 		)
-		(property "Footprint" ""
+		(property "Footprint" "DS-Resistors-SMD:CRCW0603"
 			(at 170.18 119.38 0)
 			(effects
@@
 			)
 		)
-		(property "Footprint" ""
+		(property "Footprint" "DS-Resistors-SMD:CRCW0603"
 			(at 148.59 81.28 90)
 			(effects
@@
 			)
 		)
-		(property "Footprint" ""
+		(property "Footprint" "DS-Resistors-SMD:CRCW0603"
 			(at 198.12 119.38 0)
 			(effects
@@
 			)
 		)
-		(property "Footprint" ""
+		(property "Footprint" "DS-Capacitors-SMD:MLCC0603"
 			(at 139.7 120.015 0)
 			(effects
@@
 			)
 		)
-		(property "Footprint" ""
+		(property "Footprint" "DS-Capacitors-SMD:MLCC0603"
 			(at 54.61 67.945 0)
 			(effects
@@
 	)
 	(symbol
-		(lib_name "DS-Transistors:NMOS_SGD_PWR")
 		(lib_id "DS-Transistors:NMOS_SGD_PWR")
 		(at 190.5 125.73 0)
@@
 			)
 		)
-		(property "Footprint" ""
+		(property "Footprint" "DS-Resistors-SMD:CRCW0603"
 			(at 177.8 110.49 0)
 			(effects
@@
 			)
 		)
-		(property "Footprint" ""
+		(property "Footprint" "DS-Capacitors-SMD:MLCC0805"
 			(at 91.44 94.615 0)
 			(effects
@@
 			)
 		)
-		(property "Footprint" ""
+		(property "Footprint" "DS-Capacitors-SMD:MLCC0603"
 			(at 46.99 67.945 0)
 			(effects
@@
 	)
 	(symbol
-		(lib_name "DS-Transistors:NMOS_SGD_PWR")
 		(lib_id "DS-Transistors:NMOS_SGD_PWR")
 		(at 177.8 125.73 180)
