File: hardware/electronics/powerSupplyBoard/battery_monitor.kicad_sch (KiCad schematic)
At the start: 34 parts, among them J10 1729018, J9 S3B-XH-SM4-TB, Q2 CSD18532Q5B, Q3 CSD18532Q5B, U5 BQ76905

Commit message: updated component references and sizes
Parts:
- removed C32: 1uF, lib_fp:MLCC0805, symbol lib_sch:C_horizontal
- removed C41: 220pF, lib_fp:MLCC0603, symbol lib_sch:C
- removed R18: 100R, lib_fp:CRCW0603, symbol lib_sch:R_horizontal
- removed R22: 5K1, lib_fp:CRCW0603, symbol lib_sch:R
- added C31: 1uF, lib_fp:MLCC0603, symbol lib_sch:C_horizontal
- added C39: 220pF, lib_fp:MLCC0402, symbol lib_sch:C
- added R16: 100R, lib_fp:CRCW0402, symbol lib_sch:R_horizontal
- added R20: 5K1, lib_fp:CRCW0402, symbol lib_sch:R
- C30: renamed from C31; footprint lib_fp:MLCC0805 -> lib_fp:MLCC0603; DKPN 478-KGM21AR71A105KUCT-ND -> 478-KAM15AR71C105KTCT-ND; MPN 0805ZC105KAT2A -> KAM15AR71C105KT; Package 0805 -> 0603; Voltage Rating 10V -> 16V
- C33: renamed from C34; footprint lib_fp:MLCC0805 -> lib_fp:MLCC0603; DKPN 478-KGM21AR71H105KLCT-ND -> 478-KAM15AR71C105KTCT-ND; MPN 08055C105KAT4A -> KAM15AR71C105KT; Package 0805 -> 0603; Voltage Rating 50V -> 16V
- C38: renamed from C39; footprint lib_fp:MLCC0603 -> lib_fp:MLCC0402; DKPN 478-KGM15AR71H221KTCT-ND -> 478-KAM05AR71C221KNCT-ND; MPN KGM15AR71H221KT -> KAM05AR71C221KN; Package 0603 -> 0402; Voltage Rating 50V -> 16V
- C40: footprint lib_fp:MLCC0603 -> lib_fp:MLCC0402; DKPN 478-KGM15AR71H221KTCT-ND -> 478-KAM05AR71C221KNCT-ND; MPN KGM15AR71H221KT -> KAM05AR71C221KN; Package 0603 -> 0402; Voltage Rating 50V -> 16V
- R14: renamed from R15; footprint lib_fp:CRCW0603 -> lib_fp:CRCW0402; DKPN 541-0.0GCT-ND -> 541-CRCW04020000Z0EECT-ND; MPN CRCW06030000Z0EA -> CRCW04020000Z0EE; Package 0603 -> 0402
- R15: renamed from R16; footprint lib_fp:CRCW0603 -> lib_fp:CRCW0402; DKPN 541-100HCT-ND -> 541-100LCT-ND; MPN CRCW0603100RFKEA -> CRCW0402100RFKED; Package 0603 -> 0402; Power Rating 100mW -> 62.5mW
- R17: footprint lib_fp:CRCW0603 -> lib_fp:CRCW0402; DKPN 541-100HCT-ND -> 541-100LCT-ND; MPN CRCW0603100RFKEA -> CRCW0402100RFKED; Package 0603 -> 0402; Power Rating 100mW -> 62.5mW
- R19: renamed from R20; footprint lib_fp:CRCW0603 -> lib_fp:CRCW0402; DKPN 541-10MGCT-ND -> 541-10MJCT-ND; MPN CRCW060310M0JNEA -> CRCW040210M0JNED; Power Rating 100mW -> 62.5mW
- R21: footprint lib_fp:CRCW0603 -> lib_fp:CRCW0402; DKPN 541-5.10KHCT-ND -> 541-5.10KLCT-ND; MPN CRCW06035K10FKEA -> CRCW04025K10FKED; Package 0603 -> 0402; Power Rating 100mW -> 62.5mW
- R22: renamed from R23; footprint lib_fp:CRCW0603 -> lib_fp:CRCW0402; DKPN 541-10MGCT-ND -> 541-10MJCT-ND; MPN CRCW060310M0JNEA -> CRCW040210M0JNED; Package 0603 -> 0402; Power Rating 100mW -> 62.5mW
- R23: renamed from R24; footprint lib_fp:CRCW0603 -> lib_fp:CRCW0402; DKPN 541-10KGCT-ND -> 541-10KJCT-ND; MPN CRCW060310K0JNEA -> CRCW040210K0JNED; Package 0603 -> 0402; Power Rating 100mW -> 62.5mW
- renumbered C33 to C32, C35 to C34, C36 to C35, C37 to C36, C38 to C37, R19 to R18, R25 to R24, R26 to R25, R27 to R26
Connections:
- net CHG: now also R21.1
- net DSG: now also R20.1; no longer R21.1
- net GND: now also C31.1, C39.2
- net REGSRC: now also C31.2
- net SENSE+: now also R16.2; no longer R17.2
- net SENSE-: now also R17.2
- net VC0: now also C40.1
- net VC1: now also C39.1; no longer C40.1
- net at D4.2, Q3.4, R22.1: now also R21.2
- net at C34.1, C35.1, U5.6 (SRP): now also R16.1; no longer R17.1
- net at C34.2, C35.2, U5.7 (SRN): now also R17.1
- net at Q2.4, R19.1: now also R20.2; no longer R21.2
