File: hardware/electronics/powerSupplyBoard/voltage-regulator.kicad_sch (KiCad schematic)
At the start: 9 parts, among them J7 1729018, U5 TPS62993-Q1

Commit message: fixed ERC
Connections:
- net PACK+ renamed VSYS
- net PACK- renamed GND

Commit message: changes from design review
Parts:
- removed R37: 100K, lib_fp:CRCW0402, symbol lib_sch:R
Connections:
- no-connect marks 0 -> 1
Changed lines of the file:
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@@
 		(color 0 0 0 0)
 	)
+	(no_connect
+		(at 149.86 107.95)
+	)
 	(wire
 		(pts
@@
 	(wire
 		(pts
-			(xy 165.1 105.41) (xy 165.1 107.95)
-		)
-		(stroke
-			(width 0)
-			(type default)
-		)
-	)
-	(wire
-		(pts
 			(xy 127 102.87) (xy 127 97.79)
 		)
@@
 	(wire
 		(pts
-			(xy 165.1 97.79) (xy 165.1 100.33)
-		)
-		(stroke
-			(width 0)
-			(type default)
-		)
-	)
-	(wire
-		(pts
 			(xy 129.54 118.11) (xy 124.46 118.11)
 		)
@@
 		(pts
 			(xy 101.6 97.79) (xy 127 97.79)
-		)
-		(stroke
-			(width 0)
-			(type default)
-		)
-	)
-	(wire
-		(pts
-			(xy 165.1 107.95) (xy 149.86 107.95)
 		)
 		(stroke
@@
 					(unit 1)
 				)
-			)
-		)
-	)
-	(symbol
-		(lib_id "lib_sch:R")
-		(at 165.1 102.87 0)
-		(unit 1)
-		(exclude_from_sim no)
-		(in_bom yes)
-		(on_board yes)
-		(dnp no)
-		(property "Reference" "R37"
-			(at 166.37 100.33 0)
-			(do_not_autoplace yes)
-			(effects
-				(font
-					(size 1.016 1.016)
-				)
-				(justify left)
-			)
-		)
-		(property "Value" "100K"
-			(at 166.37 101.6 0)
-			(do_not_autoplace yes)
-			(effects
-				(font
-					(size 1.016 1.016)
-				)
-				(justify left)
-			)
-		)
-		(property "Footprint" "lib_fp:CRCW0402"
-			(at 165.1 100.33 0)
-			(effects
-				(font
-					(size 1.27 1.27)
-				)
-				(hide yes)
-			)
-		)
-		(property "Datasheet" "datasheets/Vishay-Dale-DRCWe3.pdf"
-			(at 165.1 100.33 0)
-			(effects
-				(font
-					(size 1.27 1.27)
-				)
-				(hide yes)
-			)
-		)
-		(property "Description" "RES SMD 100K OHM 1% 1/16W 0402"
-			(at 165.1 102.87 0)
-			(effects
-				(font
-					(size 1.27 1.27)
-				)
-				(hide yes)
-			)
-		)
-		(property "Manufacturer" "Vishay Dale"
-			(at 165.1 100.33 0)
-			(effects
-				(font
-					(size 1.27 1.27)
-				)
-				(hide yes)
-			)
-		)
-		(property "MPN" "CRCW0402100KFKED"
-			(at 165.1 100.33 0)
-			(effects
-				(font
-					(size 1.27 1.27)
-				)
-				(hide yes)
-			)
-		)
-		(property "DKPN" "541-100KLCT-ND"
-			(at 165.1 102.87 0)
-			(effects
-				(font
-					(size 1.27 1.27)
-				)
-				(hide yes)
-			)
-		)
-		(property "Tolerance" "1%"
-			(at 166.37 102.87 0)
-			(do_not_autoplace yes)
-			(effects
-				(font
-					(size 1.016 1.016)
-				)
-				(justify left)
-			)
-		)
-		(property "Power Rating" "62.5mW"
-			(at 166.37 104.14 0)
-			(do_not_autoplace yes)
-			(effects
-				(font
-					(size 1.016 1.016)
-				)
-				(justify left)
-			)
-		)
-		(property "Package" "0402"
-			(at 166.37 105.41 0)
-			(do_not_autoplace yes)
-			(effects
-				(font
-					(size 1.016 1.016)
-				)
-				(justify left)
-			)
-		)
-		(pin "1"
-		)
-		(pin "2"
-		)
-		(instances
-			(project "powerSupplyBoard"
-				(path "/6f3ae1d2-e925-4178-b812-ea14ec542b6c/70190797-7e10-4051-a1b9-803af62c45a0"
-					(reference "R37")
-					(unit 1)
-				)

Commit message: fixed design review changes (power nets)
Parts:
- L2: symbol DS-Passives:L_horizontal -> lib_sch:L_horizontal
Changed lines of the file:
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@@
+			)
+		)
+		(property "Zener Voltage" ""
+			(at 111.76 120.65 0)
+			(effects
+				(font
+					(size 1.27 1.27)
+				)
+				(hide yes)
 			)
 		)
@@
 			)
 		)
+		(property "Zener Voltage" ""
+			(at 204.47 101.6 0)
+			(effects
+				(font
+					(size 1.27 1.27)
+				)
+				(hide yes)
+			)
+		)
 		(pin "1"
 		)
@@
 			)
 		)
+		(property "Zener Voltage" ""
+			(at 160.02 120.65 0)
+			(effects
+				(font
+					(size 1.27 1.27)
+				)
+				(hide yes)
+			)
+		)
 		(pin "1"
 		)
@@
 	)
 	(symbol
-		(lib_id "DS-Power:PWR_FLAG")
+		(lib_id "lib_sch:PWR_FLAG")
 		(at 165.1 95.25 0)
 		(unit 1)
@@
 			)
 		)
+		(property "Zener Voltage" ""
+			(at 177.8 113.03 0)
+			(effects
+				(font
+					(size 1.27 1.27)
+				)
+				(hide yes)
+			)
+		)
 		(pin "1"
 		)
@@
 			)
 		)
+		(property "Zener Voltage" ""
+			(at 101.6 113.03 0)
+			(effects
+				(font
+					(size 1.27 1.27)
+				)
+				(hide yes)
+			)
+		)
 		(pin "1"
 		)
@@
 	)
 	(symbol
-		(lib_id "DS-Power:+3V3_OUT")
+		(lib_id "lib_sch:+3V3_OUT")
 		(at 177.8 95.25 0)
 		(unit 1)
@@
 	)
 	(symbol
-		(lib_id "DS-Power:VSYS")
+		(lib_id "lib_sch:VSYS")
 		(at 101.6 95.25 0)
 		(unit 1)
@@
 				)
 				(justify left)
+			)
+		)
+		(property "Zener Voltage" ""
+			(at 124.46 123.19 0)
+			(effects
+				(font
+					(size 1.27 1.27)
+				)
+				(hide yes)
 			)
 		)
@@
 	)
 	(symbol
-		(lib_id "DS-Power:+3V3_OUT")
+		(lib_id "lib_sch:+3V3_OUT")
 		(at 198.12 97.79 0)
 		(unit 1)
@@
 	)
 	(symbol
-		(lib_id "DS-Passives:L_horizontal")
+		(lib_id "lib_sch:L_horizontal")
 		(at 154.94 97.79 0)
 		(unit 1)
@@
 				)
 				(justify left)
+			)
+		)
+		(property "Zener Voltage" ""
+			(at 154.94 97.79 0)
+			(effects
+				(font
+					(size 1.27 1.27)
+				)
+				(hide yes)
 			)
 		)
@@
 			(at 139.7 107.95 0)
 			(effects
+				(font
+					(size 1.27 1.27)
+				)
+				(hide yes)
+			)
+		)
+		(property "Zener Voltage" ""
+			(at 139.7 107.95 0)
+			(effects
