File: hardware/electronics/gnssBoard/gnssBoard.kicad_pcb (KiCad board)
At the start: 4 copper layers, 22 x 36.8 mm, 54 parts, among them J1 Standoff, J2 M.2_E_Key_PCB_Edge, Q1 DMG1013TQ-7, U1 AP7361E, U2 TXS0104VxRUTR, U3 ZED-F9P, U4 OPA344

Commit message: cleaned up PCB
Parts:
- removed D5: B0540WQ, lib_fp:SOD123
- removed D6: PTVS4V5D1BLYL, lib_fp:SOD882
- removed R13: 10K, lib_fp:CRCW0402
- removed R14: 1K, lib_fp:CRCW0402
- removed R15: 100K, lib_fp:CRCW0402
- C3: value 1uF -> 47pF
- C4, C7: value 100nF -> 1uF
- C6: value 1uF -> 100nF
- C8: value 2.2uF -> 100nF
- C9: value 47pF -> 2.2uF
- D2: value LTST-C190KGKT -> B0540WQ; footprint lib_fp:LTST-0603 -> lib_fp:SOD123
- D3: value LTST-C190KRKT -> PTVS4V5D1BLYL; footprint lib_fp:LTST-0603 -> lib_fp:SOD882
- D4: value LTST-C190TBKT -> LTST-C190KRKT
- JP1, JP2: footprint lib_fp:Jumper_2_Bridged -> lib_fp:SolderJumper-2_P1.3mm_Bridged_Pad1.0x1.5mm
- R10: value 27R -> 1K
- R11: value 27R -> 10K
- R12: value 10K -> 100K
- R2: value 10K -> 1K
- R3: value 1K -> 10K
- R4: value 4K7 -> 3K3
- R5: value 4K7 -> 10R; footprint lib_fp:CRCW0402 -> lib_fp:CRCW0603
- R6: value 10K -> 100R
- R7: value 4K7 -> 27R
- R8: value 3K3 -> 10K
- R9: value 10R -> 27R; footprint lib_fp:CRCW0603 -> lib_fp:CRCW0402
- TP1: value ~ -> +3V3
- TP10: value ~ -> ANT_DET
- TP11, TP3, TP8: value ~ -> VSS
- TP2: value ~ -> +1V8
- TP4: value ~ -> SCL
- TP5: value ~ -> SDA
- TP6: value ~ -> RXD
- TP7: value ~ -> TXD
- TP9: value ~ -> PPS
- moved R9 28.1 mm to (149.0, 113.5), turned to 90 degrees
- moved R10 26.9 mm to (142.9, 87.6), turned to 180 degrees
- moved C9 23.3 mm to (135.9, 85.8), turned to 0 degrees
- moved C3 23.2 mm to (149.8, 104.5), turned to -90 degrees
- moved R6 17.7 mm to (149.8, 107.2), turned to -90 degrees
- moved R2 13.6 mm to (133.3, 114.3), turned to 180 degrees
- moved R8 12.9 mm to (148.2, 86.8), turned to -90 degrees
- moved TP3 10.5 mm to (133.6, 112.5)
- moved R11 10.2 mm to (138.9, 111.9)
- moved TP7 8.61 mm to (141.9, 114.9)
- moved C8 8.36 mm to (130.2, 92.1), turned to 90 degrees
- moved D2 7.91 mm to (138.6, 85.4)
- moved R12 7.59 mm to (140.7, 87.6), turned to 180 degrees
- moved R4 7.34 mm to (135.4, 87.2), turned to 180 degrees
- moved TP6 5.46 mm to (143.7, 114.9)
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Connections:
- net /GNSS Module/ANT_DET renamed /ANT_DET
- net /GNSS Module/SAFEBOOT_N renamed /SAFEBOOT_N
- net /GNSS Module/SCL_3V3 renamed /SCL_3V3
- net /GNSS Module/SDA_3V3 renamed /SDA_3V3
- net /GNSS Module/ZED_RXD_3V3 renamed /ZED_RXD_3V3
- net /GNSS Module/ZED_TXD_3V3 renamed /ZED_TXD_3V3
- AE1 pad 1: /GNSS Module/ANT_IN -> /ANT_IN
- C10 pad 1: /GNSS Module/ANT_SHORT_N -> /ANT_SHORT_N
- C3 pad 1: +3V3 -> /ANT_IN
- C3 pad 2: VSS -> /RF_IN
- C8 pad 1: VBAT -> +3V3
- C9 pad 1: /GNSS Module/ANT_IN -> VBAT
- C9 pad 2: /GNSS Module/RF_IN -> VSS
- D2 pad 1: Net-(D2-Pad1) -> +3V3
- D2 pad 2: Net-(J2-~{LED_1}) -> Net-(D2-Pad2)
- D3 pad 1: Net-(D3-Pad1) -> VSS
- D3 pad 2: Net-(J2-~{LED_2}) -> /ANT_IN
- D4 pad 1: Net-(D4-Pad1) -> /PPS
- J2 pad 16: Net-(J2-~{LED_2}) -> /RTK_STAT
- J2 pad 56: /W_DISABLE -> unconnected-(J2-~{W_DISABLE1}-Pad56)
- J2 pad 6: Net-(J2-~{LED_1}) -> /GEOFENCE_STAT
- JP2 pad 1: Net-(D4-Pad2) -> Net-(JP2-Pad1)
- L1 pad 1: /GNSS Module/ANT_IN -> /ANT_IN
- L1 pad 2: /GNSS Module/ANT_SHORT_N -> /ANT_SHORT_N
- Q1 pad 1: /GNSS Module/ANT_OFF -> /ANT_OFF
- R10 pad 1: /HOST_D+ -> Net-(Q1-Pad3)
- R10 pad 2: /GNSS Module/ZED_D+ -> Net-(U4-+)
- R11 pad 1: /HOST_D- -> +3V3
- R11 pad 2: /GNSS Module/ZED_D- -> Net-(U3-D_SEL)
- R12 pad 1: VCC_RF -> Net-(U4-+)
- R12 pad 2: /GNSS Module/ANT_OFF -> VSS
- R2 pad 2: Net-(U1-PG) -> Net-(D1-Pad1)
- R3 pad 1: +1V8 -> VSS
- R3 pad 2: Net-(D1-Pad1) -> Net-(U2-OE)
- R4 pad 1: Net-(D2-Pad1) -> Net-(D2-Pad2)
- R4 pad 2: +3V3 -> VBAT
- R5 pad 1: Net-(D3-Pad1) -> /ANT_SHORT_N
- R5 pad 2: +3V3 -> Net-(Q1-Pad3)
- R6 pad 1: VSS -> Net-(JP2-Pad1)
- R6 pad 2: Net-(U2-OE) -> Net-(D4-Pad2)
- R7 pad 1: /PPS -> /HOST_D+
- R7 pad 2: Net-(D4-Pad1) -> /ZED_D+
- R8 pad 1: Net-(D5-Pad2) -> VCC_RF
- R8 pad 2: VBAT -> /ANT_OFF
- R9 pad 1: /GNSS Module/ANT_SHORT_N -> /HOST_D-
- R9 pad 2: Net-(Q1-Pad3) -> /ZED_D-
- TP3 pad 1: /ZED_RXD_1V8 -> VSS
- TP4 pad 1: /ZED_TXD_1V8 -> /SCL_1V8
- TP6 pad 1: /SCL_1V8 -> /ZED_RXD_1V8
- TP7 pad 1: VSS -> /ZED_TXD_1V8
- U1 pad 7: Net-(U1-PG) -> unconnected-(U1-PG-Pad7)
- U3 pad 19: unconnected-(U3-GEOFENCE_STAT-Pad19) -> /GEOFENCE_STAT
- U3 pad 2: /GNSS Module/RF_IN -> /RF_IN
- U3 pad 20: unconnected-(U3-RTK_STAT-Pad20) -> /RTK_STAT
- U3 pad 39: /GNSS Module/ZED_D- -> /ZED_D-
- U3 pad 40: /GNSS Module/ZED_D+ -> /ZED_D+
- U3 pad 5: /GNSS Module/ANT_OFF -> /ANT_OFF
- U3 pad 6: /GNSS Module/ANT_SHORT_N -> /ANT_SHORT_N
- U4 pad 4: /GNSS Module/ANT_SHORT_N -> /ANT_SHORT_N
Routing:
- net Net-(J2-~{LED_2}): track 38.9 -> 0.00 mm, vias 3 -> 0
- net Net-(J2-~{LED_1}): track 38.4 -> 0.00 mm, vias 3 -> 0
- net /RTK_STAT: track 0.00 -> 32.4 mm, vias 0 -> 3
- net /GEOFENCE_STAT: track 0.00 -> 32.1 mm, vias 0 -> 3
- net /GNSS Module/ZED_D-: track 27.6 -> 0.00 mm, vias 2 -> 0
- net /ZED_D-: track 0.00 -> 27.1 mm, vias 0 -> 2
- net /ZED_D+: track 0.00 -> 27.1 mm, vias 0 -> 2
- net /GNSS Module/ZED_D+: track 27.0 -> 0.00 mm, vias 2 -> 0
- net /GNSS Module/ANT_SHORT_N: track 22.8 -> 0.00 mm, vias 2 -> 0
- net /ANT_SHORT_N: track 0.00 -> 22.8 mm, vias 0 -> 2
- net /GNSS Module/ANT_IN: track 21.1 -> 0.00 mm
- net /ANT_IN: track 0.00 -> 21.1 mm
- net /GNSS Module/ANT_OFF: track 18.0 -> 0.00 mm, vias 2 -> 0
- net /ANT_OFF: track 0.00 -> 18.0 mm, vias 0 -> 2
- net Net-(D2-Pad1): track 7.63 -> 0.00 mm, vias 2 -> 0
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Other:
- board text added: "2x 20°±5°"
- board text added: "Board thickness is 0.8mm 4-Layer Beveled Edge ENIG Finish w/ Hard Gold Fingers"
- board text added: "Card Edge Bevel"
- board text added: "Embry-Riddle Aeronautical University Physical Sciences Department Madison Gleydura Master's Thesis 2024-12-21"
- board text added: "Fabrication Instructions"
- board text added: "GNSS RCVR"
- board text added: "ZED-F9P"
- board text removed: "ANT"
- board text removed: "DBG"
- board text removed: "FIX"
- board text removed: "ZED-F9P GNSS M.2 E-Key Card Embry-Riddle Aeronautical University Physical Sciences Department Madison Gleydura Master's Thesis 2024-12-02"
