File: hardware/electronics/lps28dfwBreakoutBoard/lps28dfwBreakoutBoard.kicad_pcb (KiCad board)
At the start: 2 copper layers, 25.4 x 17.8 mm, 12 parts, among them J1 2005280040, U1 LPS28DFW

Commit message: updated datasheet refs
Other:
- board text added: "PCB3D_BR_lps28Breakout"
- board text added: "PCB3D_TL_lps28Breakout"
Changed lines of the file:
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@@
+		)
+	)
+	(gr_text "PCB3D_TL_lps28Breakout"
+		(at 127 99.06 0)
+		(layer "Cmts.User")
+		(effects
+			(font
+				(size 1 1)
+				(thickness 0.15)
+			)
+			(justify right bottom)
+		)
+	)
+	(gr_text "PCB3D_BR_lps28Breakout"
+		(at 152.4 116.84 0)
+		(layer "Cmts.User")
+		(effects
+			(font
+				(size 1 1)
+				(thickness 0.15)
+			)
+			(justify left bottom)
 		)
 	)
